File: RAM/TD4_RAM/Bank_switches.sch (KiCad schematic (older format))
At the start: 18 parts, among them SW1 SW_DIP_x08, SW2 SW_DIP_x08

Commit message: Added backplane connectors to all PCBs
Parts:
- R1, R10, R11, R12, R13, R14, R15, R16, R2, R3, R4, R5, R6, R7, R8, R9: footprint (none) -> Capacitor_SMD:C_0805_2012Metric
- SW1, SW2: footprint (none) -> Button_Switch_THT:SW_DIP_SPSTx08_Slide_9.78x22.5mm_W7.62mm_P2.54mm
Changed lines of the file:
@@
 F 0 "SW2" H 5600 2567 50  0000 C CNN
 F 1 "SW_DIP_x08" H 5600 2476 50  0000 C CNN
-F 2 "" H 5600 1900 50  0001 C CNN
+F 2 "Button_Switch_THT:SW_DIP_SPSTx08_Slide_9.78x22.5mm_W7.62mm_P2.54mm" H 5600 1900 50  0001 C CNN
 F 3 "" H 5600 1900 50  0001 C CNN
 	1    5600 1900
@@
 F 0 "R2" V 5543 2700 50  0000 C CNN
 F 1 "10k" V 5634 2700 50  0000 C CNN
-F 2 "" V 5680 2700 50  0001 C CNN
+F 2 "Capacitor_SMD:C_0805_2012Metric" V 5680 2700 50  0001 C CNN
 F 3 "~" H 5750 2700 50  0001 C CNN
 	1    5750 2700
@@
 F 0 "R4" V 5543 3000 50  0000 C CNN
 F 1 "10k" V 5634 3000 50  0000 C CNN
-F 2 "" V 5680 3000 50  0001 C CNN
+F 2 "Capacitor_SMD:C_0805_2012Metric" V 5680 3000 50  0001 C CNN
 F 3 "~" H 5750 3000 50  0001 C CNN
 	1    5750 3000
@@
 F 0 "R6" V 5543 3300 50  0000 C CNN
 F 1 "10k" V 5634 3300 50  0000 C CNN
-F 2 "" V 5680 3300 50  0001 C CNN
+F 2 "Capacitor_SMD:C_0805_2012Metric" V 5680 3300 50  0001 C CNN
 F 3 "~" H 5750 3300 50  0001 C CNN
 	1    5750 3300
@@
 F 0 "R8" V 5543 3600 50  0000 C CNN
 F 1 "10k" V 5634 3600 50  0000 C CNN
-F 2 "" V 5680 3600 50  0001 C CNN
+F 2 "Capacitor_SMD:C_0805_2012Metric" V 5680 3600 50  0001 C CNN
 F 3 "~" H 5750 3600 50  0001 C CNN
 	1    5750 3600
@@
 F 0 "R10" V 5543 3900 50  0000 C CNN
 F 1 "10k" V 5634 3900 50  0000 C CNN
-F 2 "" V 5680 3900 50  0001 C CNN
+F 2 "Capacitor_SMD:C_0805_2012Metric" V 5680 3900 50  0001 C CNN
 F 3 "~" H 5750 3900 50  0001 C CNN
 	1    5750 3900
@@
 F 0 "R12" V 5543 4200 50  0000 C CNN
 F 1 "10k" V 5634 4200 50  0000 C CNN
-F 2 "" V 5680 4200 50  0001 C CNN
+F 2 "Capacitor_SMD:C_0805_2012Metric" V 5680 4200 50  0001 C CNN
 F 3 "~" H 5750 4200 50  0001 C CNN
 	1    5750 4200
@@
 F 0 "R14" V 5543 4500 50  0000 C CNN
 F 1 "10k" V 5634 4500 50  0000 C CNN
-F 2 "" V 5680 4500 50  0001 C CNN
+F 2 "Capacitor_SMD:C_0805_2012Metric" V 5680 4500 50  0001 C CNN
 F 3 "~" H 5750 4500 50  0001 C CNN
 	1    5750 4500
@@
 F 0 "R16" V 5543 4800 50  0000 C CNN
 F 1 "10k" V 5634 4800 50  0000 C CNN
-F 2 "" V 5680 4800 50  0001 C CNN
+F 2 "Capacitor_SMD:C_0805_2012Metric" V 5680 4800 50  0001 C CNN
 F 3 "~" H 5750 4800 50  0001 C CNN
 	1    5750 4800
@@
 AR Path="/5C5DC063/5CBE4539" Ref="#PWR?"  Part="1"
 AR Path="/5C5DC063/5CBDCBAA/5CBE4539" Ref="#PWR?"  Part="1"
-AR Path="/5CBF05D8/5CBE4539" Ref="#PWR0155"  Part="1"
-F 0 "#PWR0155" H 4950 3500 50  0001 C CNN
+AR Path="/5CBF05D8/5CBE4539" Ref="#PWR0170"  Part="1"
+F 0 "#PWR0170" H 4950 3500 50  0001 C CNN
 F 1 "VCC" H 4967 3823 50  0000 C CNN
 F 2 "" H 4950 3650 50  0001 C CNN
@@
 F 0 "SW1" H 3100 2567 50  0000 C CNN
 F 1 "SW_DIP_x08" H 3100 2476 50  0000 C CNN
-F 2 "" H 3100 1900 50  0001 C CNN
+F 2 "Button_Switch_THT:SW_DIP_SPSTx08_Slide_9.78x22.5mm_W7.62mm_P2.54mm" H 3100 1900 50  0001 C CNN
 F 3 "" H 3100 1900 50  0001 C CNN
 	1    3100 1900
@@
 F 0 "R1" V 3043 2700 50  0000 C CNN
 F 1 "10k" V 3134 2700 50  0000 C CNN
-F 2 "" V 3180 2700 50  0001 C CNN
+F 2 "Capacitor_SMD:C_0805_2012Metric" V 3180 2700 50  0001 C CNN
 F 3 "~" H 3250 2700 50  0001 C CNN
 	1    3250 2700
@@
 F 0 "R3" V 3043 3000 50  0000 C CNN
 F 1 "10k" V 3134 3000 50  0000 C CNN
-F 2 "" V 3180 3000 50  0001 C CNN
+F 2 "Capacitor_SMD:C_0805_2012Metric" V 3180 3000 50  0001 C CNN
 F 3 "~" H 3250 3000 50  0001 C CNN
 	1    3250 3000
@@
 F 0 "R5" V 3043 3300 50  0000 C CNN
 F 1 "10k" V 3134 3300 50  0000 C CNN
-F 2 "" V 3180 3300 50  0001 C CNN
+F 2 "Capacitor_SMD:C_0805_2012Metric" V 3180 3300 50  0001 C CNN
 F 3 "~" H 3250 3300 50  0001 C CNN
 	1    3250 3300
@@
 F 0 "R7" V 3043 3600 50  0000 C CNN
 F 1 "10k" V 3134 3600 50  0000 C CNN
-F 2 "" V 3180 3600 50  0001 C CNN
+F 2 "Capacitor_SMD:C_0805_2012Metric" V 3180 3600 50  0001 C CNN
 F 3 "~" H 3250 3600 50  0001 C CNN
 	1    3250 3600
@@
 F 0 "R9" V 3043 3900 50  0000 C CNN
 F 1 "10k" V 3134 3900 50  0000 C CNN
-F 2 "" V 3180 3900 50  0001 C CNN
+F 2 "Capacitor_SMD:C_0805_2012Metric" V 3180 3900 50  0001 C CNN
 F 3 "~" H 3250 3900 50  0001 C CNN
 	1    3250 3900
@@
 F 0 "R11" V 3043 4200 50  0000 C CNN
 F 1 "10k" V 3134 4200 50  0000 C CNN
-F 2 "" V 3180 4200 50  0001 C CNN
+F 2 "Capacitor_SMD:C_0805_2012Metric" V 3180 4200 50  0001 C CNN
 F 3 "~" H 3250 4200 50  0001 C CNN
 	1    3250 4200
@@
 F 0 "R13" V 3043 4500 50  0000 C CNN
 F 1 "10k" V 3134 4500 50  0000 C CNN
-F 2 "" V 3180 4500 50  0001 C CNN
+F 2 "Capacitor_SMD:C_0805_2012Metric" V 3180 4500 50  0001 C CNN
 F 3 "~" H 3250 4500 50  0001 C CNN
 	1    3250 4500
@@
 F 0 "R15" V 3043 4800 50  0000 C CNN
 F 1 "10k" V 3134 4800 50  0000 C CNN
-F 2 "" V 3180 4800 50  0001 C CNN
+F 2 "Capacitor_SMD:C_0805_2012Metric" V 3180 4800 50  0001 C CNN
 F 3 "~" H 3250 4800 50  0001 C CNN
 	1    3250 4800
@@
 P 2450 3650
 AR Path="/5C5DC063/5CBE8130" Ref="#PWR?"  Part="1"
-AR Path="/5CBF05D8/5CBE8130" Ref="#PWR0154"  Part="1"
-F 0 "#PWR0154" H 2450 3500 50  0001 C CNN
+AR Path="/5CBF05D8/5CBE8130" Ref="#PWR0169"  Part="1"
+F 0 "#PWR0169" H 2450 3500 50  0001 C CNN
 F 1 "VCC" H 2467 3823 50  0000 C CNN
 F 2 "" H 2450 3650 50  0001 C CNN
@@
 AR Path="/5C5DC063/5CBE4542" Ref="#PWR?"  Part="1"
 AR Path="/5C5DC063/5CBDCBAA/5CBE4542" Ref="#PWR?"  Part="1"
-AR Path="/5CBF05D8/5CBE4542" Ref="#PWR0153"  Part="1"
-F 0 "#PWR0153" H 4800 1800 50  0001 C CNN
+AR Path="/5CBF05D8/5CBE4542" Ref="#PWR0168"  Part="1"
+F 0 "#PWR0168" H 4800 1800 50  0001 C CNN
 F 1 "GND" H 4805 1877 50  0000 C CNN
 F 2 "" H 4800 2050 50  0001 C CNN
@@
 P 2300 2050
 AR Path="/5C5DC063/5CBE8139" Ref="#PWR?"  Part="1"
-AR Path="/5CBF05D8/5CBE8139" Ref="#PWR0152"  Part="1"
-F 0 "#PWR0152" H 2300 1800 50  0001 C CNN
+AR Path="/5CBF05D8/5CBE8139" Ref="#PWR0167"  Part="1"
+F 0 "#PWR0167" H 2300 1800 50  0001 C CNN
 F 1 "GND" H 2305 1877 50  0000 C CNN
 F 2 "" H 2300 2050 50  0001 C CNN

Commit message: Main RAM blocks routed
Changed lines of the file:
@@
 	5350 4800 5600 4800
-Wire Wire Line
-	5200 1800 5200 1850
 Wire Wire Line
 	5200 1900 5200 2000
@@
 	5350 4500 5350 4800
 Wire Wire Line
-	5200 1850 4800 1850
-Wire Wire Line
 	4950 3750 4950 3650
-Connection ~ 5200 1850
-Wire Wire Line
-	5200 1850 5200 1900
 $Comp
 L power:VCC #PWR?
@@
 AR Path="/5C5DC063/5CBE4539" Ref="#PWR?"  Part="1"
 AR Path="/5C5DC063/5CBDCBAA/5CBE4539" Ref="#PWR?"  Part="1"
-AR Path="/5CBF05D8/5CBE4539" Ref="#PWR0170"  Part="1"
-F 0 "#PWR0170" H 4950 3500 50  0001 C CNN
+AR Path="/5CBF05D8/5CBE4539" Ref="#PWR0173"  Part="1"
+F 0 "#PWR0173" H 4950 3500 50  0001 C CNN
 F 1 "VCC" H 4967 3823 50  0000 C CNN
 F 2 "" H 4950 3650 50  0001 C CNN
@@
 	2850 4800 3100 4800
 Wire Wire Line
-	2700 1800 2700 1850
-Wire Wire Line
 	2700 1900 2700 2000
 Wire Wire Line
@@
 	2850 4500 2850 4800
 Wire Wire Line
-	2700 1850 2300 1850
-Wire Wire Line
 	2450 3750 2450 3650
-Connection ~ 2700 1850
-Wire Wire Line
-	2700 1850 2700 1900
 $Comp
 L power:VCC #PWR?
@@
 P 2450 3650
 AR Path="/5C5DC063/5CBE8130" Ref="#PWR?"  Part="1"
-AR Path="/5CBF05D8/5CBE8130" Ref="#PWR0169"  Part="1"
-F 0 "#PWR0169" H 2450 3500 50  0001 C CNN
+AR Path="/5CBF05D8/5CBE8130" Ref="#PWR0172"  Part="1"
+F 0 "#PWR0172" H 2450 3500 50  0001 C CNN
 F 1 "VCC" H 2467 3823 50  0000 C CNN
 F 2 "" H 2450 3650 50  0001 C CNN
@@
 Text Label 6100 2200 2    50   ~ 0
 O15
-Wire Wire Line
-	4800 1850 4800 2050
-$Comp
-L power:GND #PWR?
-U 1 1 5CBE4542
-P 4800 2050
-AR Path="/5C5DC063/5CBE4542" Ref="#PWR?"  Part="1"
-AR Path="/5C5DC063/5CBDCBAA/5CBE4542" Ref="#PWR?"  Part="1"
-AR Path="/5CBF05D8/5CBE4542" Ref="#PWR0168"  Part="1"
-F 0 "#PWR0168" H 4800 1800 50  0001 C CNN
-F 1 "GND" H 4805 1877 50  0000 C CNN
-F 2 "" H 4800 2050 50  0001 C CNN
-F 3 "" H 4800 2050 50  0001 C CNN
-	1    4800 2050
-	1    0    0    -1
-$EndComp
-Wire Wire Line
-	2300 1850 2300 2050
-$Comp
-L power:GND #PWR?
-U 1 1 5CBE8139
-P 2300 2050
-AR Path="/5C5DC063/5CBE8139" Ref="#PWR?"  Part="1"
-AR Path="/5CBF05D8/5CBE8139" Ref="#PWR0167"  Part="1"
-F 0 "#PWR0167" H 2300 1800 50  0001 C CNN
-F 1 "GND" H 2305 1877 50  0000 C CNN
-F 2 "" H 2300 2050 50  0001 C CNN
-F 3 "" H 2300 2050 50  0001 C CNN
-	1    2300 2050
-	1    0    0    -1
-$EndComp
 Text Label 3600 2700 2    50   ~ 0
 O0
@@
 Text Label 6100 4800 2    50   ~ 0
 O15
+Wire Wire Line
+	5200 1800 5200 1900
+Wire Wire Line
+	5200 2200 5200 2300
+Connection ~ 5200 2200
+$Comp
+L power:GND #PWR0171
+U 1 1 5C7242CE
+P 5200 2300
+F 0 "#PWR0171" H 5200 2050 50  0001 C CNN
+F 1 "GND" H 5205 2127 50  0000 C CNN
+F 2 "" H 5200 2300 50  0001 C CNN
+F 3 "" H 5200 2300 50  0001 C CNN
+	1    5200 2300
+	1    0    0    -1
+$EndComp
+Wire Wire Line
+	2700 2200 2700 2300
+$Comp
+L power:GND #PWR0170
+U 1 1 5C7243BF
+P 2700 2300
+F 0 "#PWR0170" H 2700 2050 50  0001 C CNN
+F 1 "GND" H 2705 2127 50  0000 C CNN
+F 2 "" H 2700 2300 50  0001 C CNN
+F 3 "" H 2700 2300 50  0001 C CNN
+	1    2700 2300
+	1    0    0    -1
+$EndComp
+Wire Wire Line
+	2700 1800 2700 1900
 Wire Bus Line
 	3700 1600 3700 5300
 Wire Bus Line
 	6200 1600 6200 5300
+Connection ~ 2700 2200
 $EndSCHEMATC
