File: RAM/TD4_RAM/Memory_block.sch (KiCad schematic (older format))
At the start: 12 parts

Commit message: RAM done (sort of)
Connections:
- net CS renamed nCS
- net nQ0: no longer names the net of U?.14 (~Q)
- net nQ1: no longer names the net of U?.14 (~Q)
- net nQ2: no longer names the net of U?.14 (~Q)
- net nQ3: no longer names the net of U?.14 (~Q)
- no-connect marks 0 -> 4
Changed lines of the file:
@@
 $Descr A4 11693 8268
 encoding utf-8
-Sheet 2 20
+Sheet 20 20
 Title ""
 Date ""
@@
 RW
 Text HLabel 2000 4250 0    50   Input ~ 0
-CS
+nCS
 Wire Wire Line
 	5350 1650 5600 1650
-Wire Wire Line
-	5350 1750 5600 1750
 Entry Wire Line
 	5600 1650 5700 1750
-Entry Wire Line
-	5600 1750 5700 1850
 Text Label 5400 1650 0    50   ~ 0
 Q0
-Text Label 5400 1750 0    50   ~ 0
-nQ0
 Wire Wire Line
 	5350 3250 5600 3250
-Wire Wire Line
-	5350 3350 5600 3350
 Entry Wire Line
 	5600 3250 5700 3350
-Entry Wire Line
-	5600 3350 5700 3450
 Text Label 5400 3250 0    50   ~ 0
 Q1
-Text Label 5400 3350 0    50   ~ 0
-nQ1
 Wire Wire Line
 	5350 4850 5600 4850
-Wire Wire Line
-	5350 4950 5600 4950
 Entry Wire Line
 	5600 4850 5700 4950
-Entry Wire Line
-	5600 4950 5700 5050
 Text Label 5400 4850 0    50   ~ 0
 Q2
-Text Label 5400 4950 0    50   ~ 0
-nQ2
 Wire Wire Line
 	5350 6450 5600 6450
-Wire Wire Line
-	5350 6550 5600 6550
 Entry Wire Line
 	5600 6450 5700 6550
-Entry Wire Line
-	5600 6550 5700 6650
 Text Label 5400 6450 0    50   ~ 0
 Q3
-Text Label 5400 6550 0    50   ~ 0
-nQ3
 Wire Bus Line
 	5700 1200 7100 1200
@@
 Entry Wire Line
 	7100 3300 7200 3400
-Entry Wire Line
-	7100 3550 7200 3650
-Entry Wire Line
-	7100 3650 7200 3750
-Entry Wire Line
-	7100 3750 7200 3850
-Entry Wire Line
-	7100 3850 7200 3950
-Entry Wire Line
-	7100 3850 7200 3950
-Entry Wire Line
-	7100 3550 7200 3650
 Wire Wire Line
 	7200 3100 7600 3100
@@
 Wire Wire Line
 	7200 3400 7600 3400
-Wire Wire Line
-	7200 3650 7600 3650
-Wire Wire Line
-	7200 3750 7600 3750
-Wire Wire Line
-	7200 3850 7600 3850
-Wire Wire Line
-	7200 3950 7600 3950
 Text Label 7300 3100 0    50   ~ 0
 Q0
@@
 Text Label 7300 3400 0    50   ~ 0
 Q3
-Text Label 7300 3650 0    50   ~ 0
-nQ0
-Text Label 7300 3750 0    50   ~ 0
-nQ1
-Text Label 7300 3850 0    50   ~ 0
-nQ2
-Text Label 7300 3950 0    50   ~ 0
-nQ3
 Text HLabel 7600 3100 2    50   Output ~ 0
 Q0
@@
 Text HLabel 7600 3400 2    50   Output ~ 0
 Q3
-Text HLabel 7600 3650 2    50   Output ~ 0
-nQ0
-Text HLabel 7600 3750 2    50   Output ~ 0
-nQ1
-Text HLabel 7600 3850 2    50   Output ~ 0
-nQ2
-Text HLabel 7600 3950 2    50   Output ~ 0
-nQ3
 $Comp
 L Device:C C?
@@
 Text Notes 8100 4550 0    100  ~ 0
 Decoupling
+NoConn ~ 5350 1750
+NoConn ~ 5350 3350
+NoConn ~ 5350 4950
+NoConn ~ 5350 6550
 Wire Bus Line
-	7100 1200 7100 3850
+	7100 1200 7100 3300
 Wire Bus Line
-	5700 1200 5700 6650
+	5700 1200 5700 6550
 Wire Bus Line
 	2450 2600 2450 7300

Commit message: RAM refactoring goes on
Parts:
- gave numbers to parts that had none: 8
Connections:
- net nCS renamed ~CS
Other:
- note added: "Data inputs"
- note removed: "Data bus"
- note removed: "Data outputs\n"

Commit message: RAM done (damn buses\!)
Parts:
- renumbered C55 to C52, C56 to C53, C57 to C54, C58 to C55, U56 to U53, U57 to U54, U58 to U55, U59 to U56
Changed lines of the file:
@@
 $Descr A4 11693 8268
 encoding utf-8
-Sheet 20 46
+Sheet 44 47
 Title "TD4 RAM module"
 Date ""
@@
 $EndDescr
 $Comp
-L Custom_Symbols:К561РУ2 U56
+L Custom_Symbols:К561РУ2 U53
 U 2 1 5C5CC81A
 P 7350 5600
-F 0 "U56" H 7200 6350 100 0000 L CNN
+F 0 "U53" H 7200 6350 100 0000 L CNN
 F 1 "К561РУ2" H 7050 6200 100 0000 L CNN
 F 2 "Package_DIP:DIP-16_W7.62mm_Socket_LongPads" H 7350 4900 100 0001 C CNN
@@
 $EndComp
 $Comp
-L Custom_Symbols:К561РУ2 U56
+L Custom_Symbols:К561РУ2 U53
 U 1 1 5C5CCA5F
 P 4850 1700
-F 0 "U56" H 4850 2587 100 0000 C CNN
+F 0 "U53" H 4850 2587 100 0000 C CNN
 F 1 "К561РУ2" H 4850 2421 100 0000 C CNN
 F 2 "Package_DIP:DIP-16_W7.62mm_Socket_LongPads" H 4850 1000 100 0001 C CNN
@@
 $EndComp
 $Comp
-L Custom_Symbols:К561РУ2 U57
+L Custom_Symbols:К561РУ2 U54
 U 1 1 5C5CCAE5
 P 4850 3300
-F 0 "U57" H 4850 4187 100 0000 C CNN
+F 0 "U54" H 4850 4187 100 0000 C CNN
 F 1 "К561РУ2" H 4850 4021 100 0000 C CNN
 F 2 "Package_DIP:DIP-16_W7.62mm_Socket_LongPads" H 4850 2600 100 0001 C CNN
@@
 $EndComp
 $Comp
-L Custom_Symbols:К561РУ2 U58
+L Custom_Symbols:К561РУ2 U55
 U 1 1 5C5CCB4B
 P 4850 4900
-F 0 "U58" H 4850 5787 100 0000 C CNN
+F 0 "U55" H 4850 5787 100 0000 C CNN
 F 1 "К561РУ2" H 4850 5621 100 0000 C CNN
 F 2 "Package_DIP:DIP-16_W7.62mm_Socket_LongPads" H 4850 4200 100 0001 C CNN
@@
 $EndComp
 $Comp
-L Custom_Symbols:К561РУ2 U59
+L Custom_Symbols:К561РУ2 U56
 U 1 1 5C5CCBCB
 P 4850 6500
-F 0 "U59" H 4850 7387 100 0000 C CNN
+F 0 "U56" H 4850 7387 100 0000 C CNN
 F 1 "К561РУ2" H 4850 7221 100 0000 C CNN
 F 2 "Package_DIP:DIP-16_W7.62mm_Socket_LongPads" H 4850 5800 100 0001 C CNN
@@
 Wire Bus Line
 	4050 7300 2450 7300
-Text Label 2100 4150 0    50   ~ 0
+Text Label 1600 4150 0    50   ~ 0
 RW
-Text Label 2100 4250 0    50   ~ 0
+Text Label 1600 4250 0    50   ~ 0
 CS
-Text HLabel 2000 4150 0    50   Input ~ 0
+Text HLabel 1500 4150 0    50   Input ~ 0
 RW
-Text HLabel 2000 4250 0    50   Input ~ 0
+Text HLabel 1500 4250 0    50   Input ~ 0
 ~CS
 Wire Wire Line
@@
 	5700 1200 7100 1200
 $Comp
-L Device:C C55
+L Device:C C52
 U 1 1 5C5F9413
 P 7550 5600
-F 0 "C55" H 7665 5646 50  0000 L CNN
+F 0 "C52" H 7665 5646 50  0000 L CNN
 F 1 "100n" H 7665 5555 50  0000 L CNN
 F 2 "" H 7588 5450 50  0001 C CNN
@@
 $EndComp
 $Comp
-L Custom_Symbols:К561РУ2 U57
+L Custom_Symbols:К561РУ2 U54
 U 2 1 5C5F94AB
 P 8050 5600
-F 0 "U57" H 7900 6350 100 0000 L CNN
+F 0 "U54" H 7900 6350 100 0000 L CNN
 F 1 "К561РУ2" H 7750 6200 100 0000 L CNN
 F 2 "Package_DIP:DIP-16_W7.62mm_Socket_LongPads" H 8050 4900 100 0001 C CNN
@@
 $EndComp
 $Comp
-L Device:C C56
+L Device:C C53
 U 1 1 5C5F94B2
 P 8250 5600
-F 0 "C56" H 8365 5646 50  0000 L CNN
+F 0 "C53" H 8365 5646 50  0000 L CNN
 F 1 "100n" H 8365 5555 50  0000 L CNN
 F 2 "" H 8288 5450 50  0001 C CNN
@@
 $EndComp
 $Comp
-L Custom_Symbols:К561РУ2 U58
+L Custom_Symbols:К561РУ2 U55
 U 2 1 5C5FC441
 P 8750 5600
-F 0 "U58" H 8600 6350 100 0000 L CNN
+F 0 "U55" H 8600 6350 100 0000 L CNN
 F 1 "К561РУ2" H 8450 6200 100 0000 L CNN
 F 2 "Package_DIP:DIP-16_W7.62mm_Socket_LongPads" H 8750 4900 100 0001 C CNN
@@
 $EndComp
 $Comp
-L Device:C C57
+L Device:C C54
 U 1 1 5C5FC448
 P 8950 5600
-F 0 "C57" H 9065 5646 50  0000 L CNN
+F 0 "C54" H 9065 5646 50  0000 L CNN
 F 1 "100n" H 9065 5555 50  0000 L CNN
 F 2 "" H 8988 5450 50  0001 C CNN
@@
 $EndComp
 $Comp
-L Custom_Symbols:К561РУ2 U59
+L Custom_Symbols:К561РУ2 U56
 U 2 1 5C5FF407
 P 9450 5600
-F 0 "U59" H 9300 6350 100 0000 L CNN
+F 0 "U56" H 9300 6350 100 0000 L CNN
 F 1 "К561РУ2" H 9150 6200 100 0000 L CNN
 F 2 "Package_DIP:DIP-16_W7.62mm_Socket_LongPads" H 9450 4900 100 0001 C CNN
@@
 $EndComp
 $Comp
-L Device:C C58
+L Device:C C55
 U 1 1 5C5FF40E
 P 9650 5600
-F 0 "C58" H 9765 5646 50  0000 L CNN
+F 0 "C55" H 9765 5646 50  0000 L CNN
 F 1 "100n" H 9765 5555 50  0000 L CNN
 F 2 "" H 9688 5450 50  0001 C CNN
@@
 	7550 5100 8050 5100
 $Comp
-L power:VCC #PWR0165
+L power:VCC #PWR0156
 U 1 1 5C631C3D
 P 8450 4850
-F 0 "#PWR0165" H 8450 4700 50  0001 C CNN
+F 0 "#PWR0156" H 8450 4700 50  0001 C CNN
 F 1 "VCC" H 8467 5023 50  0000 C CNN
 F 2 "" H 8450 4850 50  0001 C CNN
@@
 	8450 5100 8750 5100
 $Comp
-L power:GND #PWR0166
+L power:GND #PWR0157
 U 1 1 5C635BF7
 P 8450 6300
-F 0 "#PWR0166" H 8450 6050 50  0001 C CNN
+F 0 "#PWR0157" H 8450 6050 50  0001 C CNN
 F 1 "GND" H 8455 6127 50  0000 C CNN
 F 2 "" H 8450 6300 50  0001 C CNN
@@
 	4000 6800 4350 6800
 Wire Wire Line
-	2000 4150 2100 4150
-Wire Wire Line
-	2000 4250 2100 4250
+	1500 4150 1600 4150
+Wire Wire Line
+	1500 4250 1600 4250
 Wire Bus Line
 	2450 3600 2450 7300
@@
 	7100 1200 7100 3300
 Text HLabel 1500 3100 0    50   Input ~ 0
-Data_in
+Data_in[0..3]
 Text HLabel 1500 3600 0    50   Input ~ 0
-Adr
+Adr[0..7]
 Text Label 1550 3100 0    50   ~ 0
 D[0..3]
 Text Label 1550 3600 0    50   ~ 0
-A[0..3]
+A[0..7]
 Wire Bus Line
 	7100 3300 7700 3300
-Wire Bus Line
-	5700 1200 5700 6550
-Wire Bus Line
-	3900 1900 3900 7150
-Wire Bus Line
-	4050 1050 4050 7300
 Text HLabel 7700 3300 2    50   Output ~ 0
-Data_out
+Data_out[0..3]
 Text Label 7350 3300 0    50   ~ 0
 Q[0..3]
+Wire Bus Line
+	5700 1200 5700 6550
+Wire Bus Line
+	3900 1900 3900 7150
+Wire Bus Line
+	4050 1050 4050 7300
 $EndSCHEMATC

Commit message: Added backplane connectors to all PCBs
Parts:
- C53: renamed from C52; footprint (none) -> Capacitor_SMD:C_0805_2012Metric
- C54: renamed from C53; footprint (none) -> Capacitor_SMD:C_0805_2012Metric
- C55: renamed from C54; footprint (none) -> Capacitor_SMD:C_0805_2012Metric
- C56: renamed from C55; footprint (none) -> Capacitor_SMD:C_0805_2012Metric
Changed lines of the file:
@@
 $Descr A4 11693 8268
 encoding utf-8
-Sheet 44 47
+Sheet 47 47
 Title "TD4 RAM module"
 Date ""
@@
 	5700 1200 7100 1200
 $Comp
-L Device:C C52
+L Device:C C53
 U 1 1 5C5F9413
 P 7550 5600
-F 0 "C52" H 7665 5646 50  0000 L CNN
+F 0 "C53" H 7665 5646 50  0000 L CNN
 F 1 "100n" H 7665 5555 50  0000 L CNN
-F 2 "" H 7588 5450 50  0001 C CNN
+F 2 "Capacitor_SMD:C_0805_2012Metric" H 7588 5450 50  0001 C CNN
 F 3 "~" H 7550 5600 50  0001 C CNN
 	1    7550 5600
@@
 $EndComp
 $Comp
-L Device:C C53
+L Device:C C54
 U 1 1 5C5F94B2
 P 8250 5600
-F 0 "C53" H 8365 5646 50  0000 L CNN
+F 0 "C54" H 8365 5646 50  0000 L CNN
 F 1 "100n" H 8365 5555 50  0000 L CNN
-F 2 "" H 8288 5450 50  0001 C CNN
+F 2 "Capacitor_SMD:C_0805_2012Metric" H 8288 5450 50  0001 C CNN
 F 3 "~" H 8250 5600 50  0001 C CNN
 	1    8250 5600
@@
 $EndComp
 $Comp
-L Device:C C54
+L Device:C C55
 U 1 1 5C5FC448
 P 8950 5600
-F 0 "C54" H 9065 5646 50  0000 L CNN
+F 0 "C55" H 9065 5646 50  0000 L CNN
 F 1 "100n" H 9065 5555 50  0000 L CNN
-F 2 "" H 8988 5450 50  0001 C CNN
+F 2 "Capacitor_SMD:C_0805_2012Metric" H 8988 5450 50  0001 C CNN
 F 3 "~" H 8950 5600 50  0001 C CNN
 	1    8950 5600
@@
 $EndComp
 $Comp
-L Device:C C55
+L Device:C C56
 U 1 1 5C5FF40E
 P 9650 5600
-F 0 "C55" H 9765 5646 50  0000 L CNN
+F 0 "C56" H 9765 5646 50  0000 L CNN
 F 1 "100n" H 9765 5555 50  0000 L CNN
-F 2 "" H 9688 5450 50  0001 C CNN
+F 2 "Capacitor_SMD:C_0805_2012Metric" H 9688 5450 50  0001 C CNN
 F 3 "~" H 9650 5600 50  0001 C CNN
 	1    9650 5600
@@
 	7550 5100 8050 5100
 $Comp
-L power:VCC #PWR0156
+L power:VCC #PWR0171
 U 1 1 5C631C3D
 P 8450 4850
-F 0 "#PWR0156" H 8450 4700 50  0001 C CNN
+F 0 "#PWR0171" H 8450 4700 50  0001 C CNN
 F 1 "VCC" H 8467 5023 50  0000 C CNN
 F 2 "" H 8450 4850 50  0001 C CNN
@@
 	8450 5100 8750 5100
 $Comp
-L power:GND #PWR0157
+L power:GND #PWR0172
 U 1 1 5C635BF7
 P 8450 6300
-F 0 "#PWR0157" H 8450 6050 50  0001 C CNN
+F 0 "#PWR0172" H 8450 6050 50  0001 C CNN
 F 1 "GND" H 8455 6127 50  0000 C CNN
 F 2 "" H 8450 6300 50  0001 C CNN

Commit message: Main RAM blocks routed
Parts:
- renumbered C53 to C51, C54 to C52, C55 to C53, C56 to C54, U53 to U49, U54 to U50, U55 to U51, U56 to U52
Changed lines of the file:
@@
 $EndDescr
 $Comp
-L Custom_Symbols:К561РУ2 U53
+L Custom_Symbols:К561РУ2 U49
 U 2 1 5C5CC81A
 P 7350 5600
-F 0 "U53" H 7200 6350 100 0000 L CNN
+F 0 "U49" H 7200 6350 100 0000 L CNN
 F 1 "К561РУ2" H 7050 6200 100 0000 L CNN
 F 2 "Package_DIP:DIP-16_W7.62mm_Socket_LongPads" H 7350 4900 100 0001 C CNN
@@
 $EndComp
 $Comp
-L Custom_Symbols:К561РУ2 U53
+L Custom_Symbols:К561РУ2 U49
 U 1 1 5C5CCA5F
 P 4850 1700
-F 0 "U53" H 4850 2587 100 0000 C CNN
+F 0 "U49" H 4850 2587 100 0000 C CNN
 F 1 "К561РУ2" H 4850 2421 100 0000 C CNN
 F 2 "Package_DIP:DIP-16_W7.62mm_Socket_LongPads" H 4850 1000 100 0001 C CNN
@@
 $EndComp
 $Comp
-L Custom_Symbols:К561РУ2 U54
+L Custom_Symbols:К561РУ2 U50
 U 1 1 5C5CCAE5
 P 4850 3300
-F 0 "U54" H 4850 4187 100 0000 C CNN
+F 0 "U50" H 4850 4187 100 0000 C CNN
 F 1 "К561РУ2" H 4850 4021 100 0000 C CNN
 F 2 "Package_DIP:DIP-16_W7.62mm_Socket_LongPads" H 4850 2600 100 0001 C CNN
@@
 $EndComp
 $Comp
-L Custom_Symbols:К561РУ2 U55
+L Custom_Symbols:К561РУ2 U51
 U 1 1 5C5CCB4B
 P 4850 4900
-F 0 "U55" H 4850 5787 100 0000 C CNN
+F 0 "U51" H 4850 5787 100 0000 C CNN
 F 1 "К561РУ2" H 4850 5621 100 0000 C CNN
 F 2 "Package_DIP:DIP-16_W7.62mm_Socket_LongPads" H 4850 4200 100 0001 C CNN
@@
 $EndComp
 $Comp
-L Custom_Symbols:К561РУ2 U56
+L Custom_Symbols:К561РУ2 U52
 U 1 1 5C5CCBCB
 P 4850 6500
-F 0 "U56" H 4850 7387 100 0000 C CNN
+F 0 "U52" H 4850 7387 100 0000 C CNN
 F 1 "К561РУ2" H 4850 7221 100 0000 C CNN
 F 2 "Package_DIP:DIP-16_W7.62mm_Socket_LongPads" H 4850 5800 100 0001 C CNN
@@
 	5700 1200 7100 1200
 $Comp
-L Device:C C53
+L Device:C C51
 U 1 1 5C5F9413
 P 7550 5600
-F 0 "C53" H 7665 5646 50  0000 L CNN
+F 0 "C51" H 7665 5646 50  0000 L CNN
 F 1 "100n" H 7665 5555 50  0000 L CNN
 F 2 "Capacitor_SMD:C_0805_2012Metric" H 7588 5450 50  0001 C CNN
@@
 $EndComp
 $Comp
-L Custom_Symbols:К561РУ2 U54
+L Custom_Symbols:К561РУ2 U50
 U 2 1 5C5F94AB
 P 8050 5600
-F 0 "U54" H 7900 6350 100 0000 L CNN
+F 0 "U50" H 7900 6350 100 0000 L CNN
 F 1 "К561РУ2" H 7750 6200 100 0000 L CNN
 F 2 "Package_DIP:DIP-16_W7.62mm_Socket_LongPads" H 8050 4900 100 0001 C CNN
@@
 $EndComp
 $Comp
-L Device:C C54
+L Device:C C52
 U 1 1 5C5F94B2
 P 8250 5600
-F 0 "C54" H 8365 5646 50  0000 L CNN
+F 0 "C52" H 8365 5646 50  0000 L CNN
 F 1 "100n" H 8365 5555 50  0000 L CNN
 F 2 "Capacitor_SMD:C_0805_2012Metric" H 8288 5450 50  0001 C CNN
@@
 $EndComp
 $Comp
-L Custom_Symbols:К561РУ2 U55
+L Custom_Symbols:К561РУ2 U51
 U 2 1 5C5FC441
 P 8750 5600
-F 0 "U55" H 8600 6350 100 0000 L CNN
+F 0 "U51" H 8600 6350 100 0000 L CNN
 F 1 "К561РУ2" H 8450 6200 100 0000 L CNN
 F 2 "Package_DIP:DIP-16_W7.62mm_Socket_LongPads" H 8750 4900 100 0001 C CNN
@@
 $EndComp
 $Comp
-L Device:C C55
+L Device:C C53
 U 1 1 5C5FC448
 P 8950 5600
-F 0 "C55" H 9065 5646 50  0000 L CNN
+F 0 "C53" H 9065 5646 50  0000 L CNN
 F 1 "100n" H 9065 5555 50  0000 L CNN
 F 2 "Capacitor_SMD:C_0805_2012Metric" H 8988 5450 50  0001 C CNN
@@
 $EndComp
 $Comp
-L Custom_Symbols:К561РУ2 U56
+L Custom_Symbols:К561РУ2 U52
 U 2 1 5C5FF407
 P 9450 5600
-F 0 "U56" H 9300 6350 100 0000 L CNN
+F 0 "U52" H 9300 6350 100 0000 L CNN
 F 1 "К561РУ2" H 9150 6200 100 0000 L CNN
 F 2 "Package_DIP:DIP-16_W7.62mm_Socket_LongPads" H 9450 4900 100 0001 C CNN
@@
 $EndComp
 $Comp
-L Device:C C56
+L Device:C C54
 U 1 1 5C5FF40E
 P 9650 5600
-F 0 "C56" H 9765 5646 50  0000 L CNN
+F 0 "C54" H 9765 5646 50  0000 L CNN
 F 1 "100n" H 9765 5555 50  0000 L CNN
 F 2 "Capacitor_SMD:C_0805_2012Metric" H 9688 5450 50  0001 C CNN
@@
 	7550 5100 8050 5100
 $Comp
-L power:VCC #PWR0171
+L power:VCC #PWR0174
 U 1 1 5C631C3D
 P 8450 4850
-F 0 "#PWR0171" H 8450 4700 50  0001 C CNN
+F 0 "#PWR0174" H 8450 4700 50  0001 C CNN
 F 1 "VCC" H 8467 5023 50  0000 C CNN
 F 2 "" H 8450 4850 50  0001 C CNN
@@
 	8450 5100 8750 5100
 $Comp
-L power:GND #PWR0172
+L power:GND #PWR0175
 U 1 1 5C635BF7
 P 8450 6300
-F 0 "#PWR0172" H 8450 6050 50  0001 C CNN
+F 0 "#PWR0175" H 8450 6050 50  0001 C CNN
 F 1 "GND" H 8455 6127 50  0000 C CNN
 F 2 "" H 8450 6300 50  0001 C CNN
