File: RAM/TD4_RAM/TD4_RAM.kicad_pcb (KiCad board)
At the start: 2 copper layers, 190 x 160 mm, 127 parts, among them J1 Conn_02x32_Row_Letter_First, SW1 SW_DIP_x08, SW2 SW_DIP_x08, U1 74AHC1G32, U10 74HC86, U11 74HC86, U12 74HC86, U13 74HC86, U14 74HC86, U15 74HC86, U16 74HC86, U17 74HC86, U18 74HC86, U19 74HC86, U2 74HC86, U20 74HC04, U21 74HC04, U22 74HC04, U23 74HC04, U24 74HC04, U25 74HC04, U26 74HC04, U27 74HC04, U28 74HC04, U29 74HC04, U3 74HC04, U30 74HC04, U31 74HC04, U32 74HC04, U33 74HC04, U34 74HC04, U35 74HC21, U36 74HC21, U37 74HC21, U38 74HC21, U39 74HC21, U4 74HC21, U40 74HC21, U41 74HC21, U42 74HC21, U43 74HC21, U44 74HC21, U45 74HC86, U46 74HC86, U47 74HC86, U48 74HC86, U49 К561РУ2, U5 74HC86, U50 К561РУ2, U51 К561РУ2, U52 К561РУ2, U6 74HC86, U7 74HC86, U8 74HC86, U9 74HC86

Commit message: RAM routing done
Parts:
- removed C57, C58: 100n, Capacitor_SMD:C_0805_2012Metric
- added REF**: MountingHole_4.3mm_M4_Pad, MountingHole:MountingHole_4.3mm_M4_Pad, F.Cu at (60.0, 170.0)
- added REF**: MountingHole_4.3mm_M4_Pad, MountingHole:MountingHole_4.3mm_M4_Pad, F.Cu at (230.0, 170.0)
- added REF**: MountingHole_4.3mm_M4_Pad, MountingHole:MountingHole_4.3mm_M4_Pad, F.Cu at (230.0, 30.0)
- added REF**: MountingHole_4.3mm_M4_Pad, MountingHole:MountingHole_4.3mm_M4_Pad, F.Cu at (60.0, 30.0)
- moved C2 300.1 mm to (65.1, 61.9), turned to 90 degrees
- moved C1 290.8 mm to (61.7, 61.9), turned to 90 degrees
- moved C51 174.6 mm to (158.9, 171.6)
- moved C54 174.6 mm to (198.9, 171.6)
- moved U49 174.6 mm to (155.2, 149.9)
- moved U52 174.6 mm to (195.1, 149.9)
- moved C52 174.6 mm to (172.4, 171.6)
- moved U50 174.6 mm to (168.4, 149.9)
- moved U51 174.6 mm to (181.9, 149.9)
- moved C53 174.6 mm to (185.6, 171.6)
- moved U1 164.1 mm to (209.6, 141.7)
- moved C3 160.0 mm to (212.6, 142.7), turned to 270 degrees
- moved SW1 158.9 mm to (215.1, 133.5), turned to 180 degrees
- moved R1 140.0 mm to (203.3, 133.5), turned to 270 degrees
- moved SW2 136.5 mm to (215.1, 108.1), turned to 180 degrees
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Connections:
- U43 pad 1: Net-(U42-Pad6) -> /sheet5CBA2603/A8
- U43 pad 2: Net-(U42-Pad8) -> /sheet5CBA2603/A9
- U43 pad 4: Net-(U43-Pad4) -> /sheet5CBA2603/A10
- U43 pad 5: Net-(U43-Pad5) -> /sheet5CBA2603/A11
- U43 pad 6: /sheet5CBA2603/Q0 -> Net-(U43-Pad6)
- U43 pad 8: Net-(U43-Pad5) -> Net-(U43-Pad8)
- U44 pad 1: /sheet5CBA2603/A8 -> Net-(U42-Pad6)
- U44 pad 2: /sheet5CBA2603/A9 -> Net-(U42-Pad8)
- U44 pad 4: /sheet5CBA2603/A10 -> Net-(U43-Pad6)
- U44 pad 5: /sheet5CBA2603/A11 -> Net-(U43-Pad8)
- U44 pad 6: Net-(U43-Pad4) -> /sheet5CBA2603/Q0
Routing:
- net GND: track 1166.7 -> 1770.5 mm, vias 97 -> 121
- net VCC: track 1014.5 -> 1613.9 mm, vias 36 -> 59
- net /RAM_A4: track 119.7 -> 604.0 mm, vias 16 -> 19
- net /RAM_A5: track 136.6 -> 601.1 mm, vias 16 -> 18
- net /RAM_A6: track 412.9 -> 843.6 mm, vias 48 -> 52
- net /RAM_A7: track 421.7 -> 775.3 mm, vias 32 -> 52
- net /RAM_D3: track 2.54 -> 207.6 mm, vias 0 -> 4
- net /RAM_D2: track 2.54 -> 181.2 mm, vias 0 -> 3
- net /RAM_WE: track 0.00 -> 166.2 mm, vias 0 -> 4
- net /RAM_D1: track 2.54 -> 167.1 mm, vias 0 -> 3
- net /sheet5CBF05D3/B7: track 5.59 -> 166.8 mm, vias 1 -> 7
- net /sheet5CBF05D3/B6: track 11.4 -> 165.9 mm, vias 2 -> 8
- net /RAM_D0: track 2.54 -> 156.2 mm, vias 0 -> 3
- net /RAM_A0: track 43.0 -> 181.6 mm, vias 0 -> 3
- net /RAM_A1: track 43.0 -> 180.8 mm, vias 0 -> 3
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