File: core/TD4_core/4bit_3state_buf.sch (KiCad schematic (older format))
At the start: 2 parts, among them U34 74HC125

Commit message: Fixed minor core PCB errors
Changed lines of the file:
@@
 $Descr A4 11693 8268
 encoding utf-8
-Sheet 21 30
+Sheet 30 30
 Title "TD4 core module"
 Date ""
@@
 AR Path="/5C6C9696/5C662A4F" Ref="U?"  Part="1"
 AR Path="/5C6CE91F/5C662A4F" Ref="U?"  Part="1"
-AR Path="/5C72E552/5C7339DC/5C662A4F" Ref="U?"  Part="1"
-AR Path="/5C74C5C4/5C7339DC/5C662A4F" Ref="U?"  Part="1"
+AR Path="/5C72E552/5C7339DC/5C662A4F" Ref="U38"  Part="1"
+AR Path="/5C74C5C4/5C7339DC/5C662A4F" Ref="U39"  Part="1"
 AR Path="/5C758048/5C7339DC/5C662A4F" Ref="U?"  Part="1"
-AR Path="/5C77FFF0/5C780016/5C7339DC/5C662A4F" Ref="U?"  Part="1"
-F 0 "U34" H 5600 2567 50  0000 C CNN
+AR Path="/5C77FFF0/5C780016/5C7339DC/5C662A4F" Ref="U40"  Part="1"
+F 0 "U40" H 5600 2567 50  0000 C CNN
 F 1 "74HC125" H 5600 2476 50  0000 C CNN
 F 2 "Package_SO:SOIC-14_3.9x8.7mm_P1.27mm" H 5600 2250 50  0001 C CNN
@@
 AR Path="/5C6C9696/5C662AA5" Ref="U?"  Part="2"
 AR Path="/5C6CE91F/5C662AA5" Ref="U?"  Part="2"
-AR Path="/5C72E552/5C7339DC/5C662AA5" Ref="U?"  Part="2"
-AR Path="/5C74C5C4/5C7339DC/5C662AA5" Ref="U?"  Part="2"
+AR Path="/5C72E552/5C7339DC/5C662AA5" Ref="U38"  Part="2"
+AR Path="/5C74C5C4/5C7339DC/5C662AA5" Ref="U39"  Part="2"
 AR Path="/5C758048/5C7339DC/5C662AA5" Ref="U?"  Part="2"
-AR Path="/5C77FFF0/5C780016/5C7339DC/5C662AA5" Ref="U?"  Part="2"
-F 0 "U34" H 5600 3317 50  0000 C CNN
+AR Path="/5C77FFF0/5C780016/5C7339DC/5C662AA5" Ref="U40"  Part="2"
+F 0 "U40" H 5600 3317 50  0000 C CNN
 F 1 "74HC125" H 5600 3226 50  0000 C CNN
 F 2 "Package_SO:SOIC-14_3.9x8.7mm_P1.27mm" H 5600 3000 50  0001 C CNN
@@
 AR Path="/5C6C9696/5C662AD3" Ref="U?"  Part="3"
 AR Path="/5C6CE91F/5C662AD3" Ref="U?"  Part="3"
-AR Path="/5C72E552/5C7339DC/5C662AD3" Ref="U?"  Part="3"
-AR Path="/5C74C5C4/5C7339DC/5C662AD3" Ref="U?"  Part="3"
+AR Path="/5C72E552/5C7339DC/5C662AD3" Ref="U38"  Part="3"
+AR Path="/5C74C5C4/5C7339DC/5C662AD3" Ref="U39"  Part="3"
 AR Path="/5C758048/5C7339DC/5C662AD3" Ref="U?"  Part="3"
-AR Path="/5C77FFF0/5C780016/5C7339DC/5C662AD3" Ref="U?"  Part="3"
-F 0 "U34" H 5600 4067 50  0000 C CNN
+AR Path="/5C77FFF0/5C780016/5C7339DC/5C662AD3" Ref="U40"  Part="3"
+F 0 "U40" H 5600 4067 50  0000 C CNN
 F 1 "74HC125" H 5600 3976 50  0000 C CNN
 F 2 "Package_SO:SOIC-14_3.9x8.7mm_P1.27mm" H 5600 3750 50  0001 C CNN
@@
 AR Path="/5C6C9696/5C662B05" Ref="U?"  Part="4"
 AR Path="/5C6CE91F/5C662B05" Ref="U?"  Part="4"
-AR Path="/5C72E552/5C7339DC/5C662B05" Ref="U?"  Part="4"
-AR Path="/5C74C5C4/5C7339DC/5C662B05" Ref="U?"  Part="4"
+AR Path="/5C72E552/5C7339DC/5C662B05" Ref="U38"  Part="4"
+AR Path="/5C74C5C4/5C7339DC/5C662B05" Ref="U39"  Part="4"
 AR Path="/5C758048/5C7339DC/5C662B05" Ref="U?"  Part="4"
-AR Path="/5C77FFF0/5C780016/5C7339DC/5C662B05" Ref="U?"  Part="4"
-F 0 "U34" H 5600 4817 50  0000 C CNN
+AR Path="/5C77FFF0/5C780016/5C7339DC/5C662B05" Ref="U40"  Part="4"
+F 0 "U40" H 5600 4817 50  0000 C CNN
 F 1 "74HC125" H 5600 4726 50  0000 C CNN
 F 2 "Package_SO:SOIC-14_3.9x8.7mm_P1.27mm" H 5600 4500 50  0001 C CNN
@@
 AR Path="/5C6C9696/5C662B31" Ref="U?"  Part="5"
 AR Path="/5C6CE91F/5C662B31" Ref="U?"  Part="5"
-AR Path="/5C72E552/5C7339DC/5C662B31" Ref="U?"  Part="5"
-AR Path="/5C74C5C4/5C7339DC/5C662B31" Ref="U?"  Part="5"
+AR Path="/5C72E552/5C7339DC/5C662B31" Ref="U38"  Part="5"
+AR Path="/5C74C5C4/5C7339DC/5C662B31" Ref="U39"  Part="5"
 AR Path="/5C758048/5C7339DC/5C662B31" Ref="U?"  Part="5"
-AR Path="/5C77FFF0/5C780016/5C7339DC/5C662B31" Ref="U?"  Part="5"
-F 0 "U34" H 8530 5746 50  0000 L CNN
+AR Path="/5C77FFF0/5C780016/5C7339DC/5C662B31" Ref="U40"  Part="5"
+F 0 "U40" H 8530 5746 50  0000 L CNN
 F 1 "74HC125" H 8530 5655 50  0000 L CNN
 F 2 "Package_SO:SOIC-14_3.9x8.7mm_P1.27mm" H 8300 5700 50  0001 C CNN
@@
 	5900 4500 6000 4500
 Text Label 5500 2550 2    50   ~ 0
-EN
+~EN
 Text Label 5500 3300 2    50   ~ 0
-EN
+~EN
 Text Label 5500 4050 2    50   ~ 0
-EN
-Text Label 5500 4800 2    50   ~ 0
-EN
+~EN
 Text Label 5200 2250 0    50   ~ 0
 A0
@@
 AR Path="/5C6C9696/5C6652A0" Ref="C?"  Part="1"
 AR Path="/5C6CE91F/5C6652A0" Ref="C?"  Part="1"
-AR Path="/5C72E552/5C7339DC/5C6652A0" Ref="C?"  Part="1"
-AR Path="/5C74C5C4/5C7339DC/5C6652A0" Ref="C?"  Part="1"
+AR Path="/5C72E552/5C7339DC/5C6652A0" Ref="C44"  Part="1"
+AR Path="/5C74C5C4/5C7339DC/5C6652A0" Ref="C45"  Part="1"
 AR Path="/5C758048/5C7339DC/5C6652A0" Ref="C?"  Part="1"
-AR Path="/5C77FFF0/5C780016/5C7339DC/5C6652A0" Ref="C?"  Part="1"
-F 0 "C40" H 9115 5746 50  0000 L CNN
+AR Path="/5C77FFF0/5C780016/5C7339DC/5C6652A0" Ref="C46"  Part="1"
+F 0 "C46" H 9115 5746 50  0000 L CNN
 F 1 "100n" H 9115 5655 50  0000 L CNN
 F 2 "Capacitor_SMD:C_0805_2012Metric" H 9038 5550 50  0001 C CNN
@@
 	9000 6300 9000 5850
 $Comp
-L power:VCC #PWR0127
+L power:VCC #PWR0129
 U 1 1 5C6657D0
 P 8650 5100
-AR Path="/5C6628C5/5C6657D0" Ref="#PWR0127"  Part="1"
+AR Path="/5C6628C5/5C6657D0" Ref="#PWR0129"  Part="1"
 AR Path="/5C6C9696/5C6657D0" Ref="#PWR?"  Part="1"
 AR Path="/5C6CE91F/5C6657D0" Ref="#PWR?"  Part="1"
-AR Path="/5C72E552/5C7339DC/5C6657D0" Ref="#PWR?"  Part="1"
-AR Path="/5C74C5C4/5C7339DC/5C6657D0" Ref="#PWR?"  Part="1"
+AR Path="/5C72E552/5C7339DC/5C6657D0" Ref="#PWR0143"  Part="1"
+AR Path="/5C74C5C4/5C7339DC/5C6657D0" Ref="#PWR0145"  Part="1"
 AR Path="/5C758048/5C7339DC/5C6657D0" Ref="#PWR?"  Part="1"
-AR Path="/5C77FFF0/5C780016/5C7339DC/5C6657D0" Ref="#PWR?"  Part="1"
-F 0 "#PWR0127" H 8650 4950 50  0001 C CNN
+AR Path="/5C77FFF0/5C780016/5C7339DC/5C6657D0" Ref="#PWR0147"  Part="1"
+F 0 "#PWR0147" H 8650 4950 50  0001 C CNN
 F 1 "VCC" H 8667 5273 50  0000 C CNN
 F 2 "" H 8650 5100 50  0001 C CNN
@@
 	8650 5100 9000 5100
 $Comp
-L power:GND #PWR0128
+L power:GND #PWR0130
 U 1 1 5C66581B
 P 8650 6300
-AR Path="/5C6628C5/5C66581B" Ref="#PWR0128"  Part="1"
+AR Path="/5C6628C5/5C66581B" Ref="#PWR0130"  Part="1"
 AR Path="/5C6C9696/5C66581B" Ref="#PWR?"  Part="1"
 AR Path="/5C6CE91F/5C66581B" Ref="#PWR?"  Part="1"
-AR Path="/5C72E552/5C7339DC/5C66581B" Ref="#PWR?"  Part="1"
-AR Path="/5C74C5C4/5C7339DC/5C66581B" Ref="#PWR?"  Part="1"
+AR Path="/5C72E552/5C7339DC/5C66581B" Ref="#PWR0144"  Part="1"
+AR Path="/5C74C5C4/5C7339DC/5C66581B" Ref="#PWR0146"  Part="1"
 AR Path="/5C758048/5C7339DC/5C66581B" Ref="#PWR?"  Part="1"
-AR Path="/5C77FFF0/5C780016/5C7339DC/5C66581B" Ref="#PWR?"  Part="1"
-F 0 "#PWR0128" H 8650 6050 50  0001 C CNN
+AR Path="/5C77FFF0/5C780016/5C7339DC/5C66581B" Ref="#PWR0148"  Part="1"
+F 0 "#PWR0148" H 8650 6050 50  0001 C CNN
 F 1 "GND" H 8655 6127 50  0000 C CNN
 F 2 "" H 8650 6300 50  0001 C CNN
@@
 	4200 2300 4300 2300
 Text Label 4300 2300 0    50   ~ 0
-EN
+~EN
+Text Label 5500 4800 2    50   ~ 0
+~EN
 Wire Bus Line
 	5100 1900 5100 4400
