File: core/TD4_core/Adder.sch (KiCad schematic (older format))
At the start: 30 parts

Commit message: RAM refactoring goes on
Connections:
- net A_0 renamed A0
- net A_1 renamed A1
- net A_2 renamed A2
- net A_3 renamed A3
- net B_0 renamed B0
- net B_1 renamed B1
- net B_2 renamed B2
- net B_3 renamed B3
- net Sum_0 renamed Q0
- net Sum_1 renamed Q1
- net Sum_2 renamed Q2
- net Sum_3 renamed Q3
Other:
- moved on the sheet: U?A, U?B, U?C, U?D

Commit message: Main core schematic done; only decoder left
Changed lines of the file:
@@
 $Descr A4 11693 8268
 encoding utf-8
-Sheet 3 6
+Sheet 3 9
 Title "TD4 core module"
 Date ""
@@
 Q[0..3]
 Text HLabel 1000 2500 0    50   Input ~ 0
-A
+A[0..3]
 Text HLabel 1000 2900 0    50   Input ~ 0
-B
+B[0..3]
 Text HLabel 10100 3200 2    50   Output ~ 0
-Q
+Q[0..3]
 $EndSCHEMATC

Commit message: Core assembled; decoder left
Parts:
- gave numbers to parts that had none: 10

Commit message: Core schematic done. Backplane connector added, including separate .sch file to append.
Parts:
- C11: renamed from C5; footprint (none) -> Capacitor_SMD:C_0805_2012Metric
- C12: renamed from C6; footprint (none) -> Capacitor_SMD:C_0805_2012Metric
- C13: renamed from C7; footprint (none) -> Capacitor_SMD:C_0805_2012Metric
- C14: renamed from C8; footprint (none) -> Capacitor_SMD:C_0805_2012Metric
- C15: renamed from C9; footprint (none) -> Capacitor_SMD:C_0805_2012Metric
- U5, U6, U7, U8, U9: footprint (none) -> Package_SO:SOIC-14_3.9x8.7mm_P1.27mm
Changed lines of the file:
@@
 F 0 "U5" H 2850 1475 50  0000 C CNN
 F 1 "74HC86" H 2850 1384 50  0000 C CNN
-F 2 "" H 2850 1150 50  0001 C CNN
+F 2 "Package_SO:SOIC-14_3.9x8.7mm_P1.27mm" H 2850 1150 50  0001 C CNN
 F 3 "http://www.ti.com/lit/gpn/sn74HC86" H 2850 1150 50  0001 C CNN
 	1    2850 1150
@@
 F 0 "U5" H 3800 1675 50  0000 C CNN
 F 1 "74HC86" H 3800 1584 50  0000 C CNN
-F 2 "" H 3800 1350 50  0001 C CNN
+F 2 "Package_SO:SOIC-14_3.9x8.7mm_P1.27mm" H 3800 1350 50  0001 C CNN
 F 3 "http://www.ti.com/lit/gpn/sn74HC86" H 3800 1350 50  0001 C CNN
 	2    3800 1350
@@
 F 0 "U5" H 1730 6946 50  0000 L CNN
 F 1 "74HC86" H 1730 6855 50  0000 L CNN
-F 2 "" H 1500 6900 50  0001 C CNN
+F 2 "Package_SO:SOIC-14_3.9x8.7mm_P1.27mm" H 1500 6900 50  0001 C CNN
 F 3 "http://www.ti.com/lit/gpn/sn74HC86" H 1500 6900 50  0001 C CNN
 	5    1500 6900
@@
 F 0 "U8" H 2930 6946 50  0000 L CNN
 F 1 "74HC86" H 2930 6855 50  0000 L CNN
-F 2 "" H 2700 6900 50  0001 C CNN
+F 2 "Package_SO:SOIC-14_3.9x8.7mm_P1.27mm" H 2700 6900 50  0001 C CNN
 F 3 "http://www.ti.com/lit/gpn/sn74HC86" H 2700 6900 50  0001 C CNN
 	5    2700 6900
@@
 F 0 "U6" H 3800 2225 50  0000 C CNN
 F 1 "74HC08" H 3800 2134 50  0000 C CNN
-F 2 "" H 3800 1900 50  0001 C CNN
+F 2 "Package_SO:SOIC-14_3.9x8.7mm_P1.27mm" H 3800 1900 50  0001 C CNN
 F 3 "http://www.ti.com/lit/gpn/sn74LS08" H 3800 1900 50  0001 C CNN
 	1    3800 1900
@@
 F 0 "U6" H 3800 2825 50  0000 C CNN
 F 1 "74HC08" H 3800 2734 50  0000 C CNN
-F 2 "" H 3800 2500 50  0001 C CNN
+F 2 "Package_SO:SOIC-14_3.9x8.7mm_P1.27mm" H 3800 2500 50  0001 C CNN
 F 3 "http://www.ti.com/lit/gpn/sn74LS08" H 3800 2500 50  0001 C CNN
 	2    3800 2500
@@
 F 0 "U9" H 4130 6946 50  0000 L CNN
 F 1 "74HC08" H 4130 6855 50  0000 L CNN
-F 2 "" H 3900 6900 50  0001 C CNN
+F 2 "Package_SO:SOIC-14_3.9x8.7mm_P1.27mm" H 3900 6900 50  0001 C CNN
 F 3 "http://www.ti.com/lit/gpn/sn74LS08" H 3900 6900 50  0001 C CNN
 	5    3900 6900
@@
 F 0 "U6" H 5330 6896 50  0000 L CNN
 F 1 "74HC08" H 5330 6805 50  0000 L CNN
-F 2 "" H 5100 6850 50  0001 C CNN
+F 2 "Package_SO:SOIC-14_3.9x8.7mm_P1.27mm" H 5100 6850 50  0001 C CNN
 F 3 "http://www.ti.com/lit/gpn/sn74LS08" H 5100 6850 50  0001 C CNN
 	5    5100 6850
@@
 F 0 "U7" H 4550 2525 50  0000 C CNN
 F 1 "74HC32" H 4550 2434 50  0000 C CNN
-F 2 "" H 4550 2200 50  0001 C CNN
+F 2 "Package_SO:SOIC-14_3.9x8.7mm_P1.27mm" H 4550 2200 50  0001 C CNN
 F 3 "http://www.ti.com/lit/gpn/sn74LS32" H 4550 2200 50  0001 C CNN
 	1    4550 2200
@@
 F 0 "U7" H 6530 6896 50  0000 L CNN
 F 1 "74HC32" H 6530 6805 50  0000 L CNN
-F 2 "" H 6300 6850 50  0001 C CNN
+F 2 "Package_SO:SOIC-14_3.9x8.7mm_P1.27mm" H 6300 6850 50  0001 C CNN
 F 3 "http://www.ti.com/lit/gpn/sn74LS32" H 6300 6850 50  0001 C CNN
 	5    6300 6850
@@
 F 0 "U5" H 6800 1475 50  0000 C CNN
 F 1 "74HC86" H 6800 1384 50  0000 C CNN
-F 2 "" H 6800 1150 50  0001 C CNN
+F 2 "Package_SO:SOIC-14_3.9x8.7mm_P1.27mm" H 6800 1150 50  0001 C CNN
 F 3 "http://www.ti.com/lit/gpn/sn74HC86" H 6800 1150 50  0001 C CNN
 	3    6800 1150
@@
 F 0 "U5" H 7750 1675 50  0000 C CNN
 F 1 "74HC86" H 7750 1584 50  0000 C CNN
-F 2 "" H 7750 1350 50  0001 C CNN
+F 2 "Package_SO:SOIC-14_3.9x8.7mm_P1.27mm" H 7750 1350 50  0001 C CNN
 F 3 "http://www.ti.com/lit/gpn/sn74HC86" H 7750 1350 50  0001 C CNN
 	4    7750 1350
@@
 F 0 "U6" H 7750 2225 50  0000 C CNN
 F 1 "74HC08" H 7750 2134 50  0000 C CNN
-F 2 "" H 7750 1900 50  0001 C CNN
+F 2 "Package_SO:SOIC-14_3.9x8.7mm_P1.27mm" H 7750 1900 50  0001 C CNN
 F 3 "http://www.ti.com/lit/gpn/sn74LS08" H 7750 1900 50  0001 C CNN
 	3    7750 1900
@@
 F 0 "U6" H 7750 2825 50  0000 C CNN
 F 1 "74HC08" H 7750 2734 50  0000 C CNN
-F 2 "" H 7750 2500 50  0001 C CNN
+F 2 "Package_SO:SOIC-14_3.9x8.7mm_P1.27mm" H 7750 2500 50  0001 C CNN
 F 3 "http://www.ti.com/lit/gpn/sn74LS08" H 7750 2500 50  0001 C CNN
 	4    7750 2500
@@
 F 0 "U7" H 8500 2525 50  0000 C CNN
 F 1 "74HC32" H 8500 2434 50  0000 C CNN
-F 2 "" H 8500 2200 50  0001 C CNN
+F 2 "Package_SO:SOIC-14_3.9x8.7mm_P1.27mm" H 8500 2200 50  0001 C CNN
 F 3 "http://www.ti.com/lit/gpn/sn74LS32" H 8500 2200 50  0001 C CNN
 	2    8500 2200
@@
 F 0 "U8" H 2850 3975 50  0000 C CNN
 F 1 "74HC86" H 2850 3884 50  0000 C CNN
-F 2 "" H 2850 3650 50  0001 C CNN
+F 2 "Package_SO:SOIC-14_3.9x8.7mm_P1.27mm" H 2850 3650 50  0001 C CNN
 F 3 "http://www.ti.com/lit/gpn/sn74HC86" H 2850 3650 50  0001 C CNN
 	1    2850 3650
@@
 F 0 "U8" H 3750 4175 50  0000 C CNN
 F 1 "74HC86" H 3750 4084 50  0000 C CNN
-F 2 "" H 3750 3850 50  0001 C CNN
+F 2 "Package_SO:SOIC-14_3.9x8.7mm_P1.27mm" H 3750 3850 50  0001 C CNN
 F 3 "http://www.ti.com/lit/gpn/sn74HC86" H 3750 3850 50  0001 C CNN
 	2    3750 3850
@@
 F 0 "U9" H 3750 4725 50  0000 C CNN
 F 1 "74HC08" H 3750 4634 50  0000 C CNN
-F 2 "" H 3750 4400 50  0001 C CNN
+F 2 "Package_SO:SOIC-14_3.9x8.7mm_P1.27mm" H 3750 4400 50  0001 C CNN
 F 3 "http://www.ti.com/lit/gpn/sn74LS08" H 3750 4400 50  0001 C CNN
 	1    3750 4400
@@
 F 0 "U9" H 3750 5325 50  0000 C CNN
 F 1 "74HC08" H 3750 5234 50  0000 C CNN
-F 2 "" H 3750 5000 50  0001 C CNN
+F 2 "Package_SO:SOIC-14_3.9x8.7mm_P1.27mm" H 3750 5000 50  0001 C CNN
 F 3 "http://www.ti.com/lit/gpn/sn74LS08" H 3750 5000 50  0001 C CNN
 	2    3750 5000
@@
 F 0 "U7" H 4500 5025 50  0000 C CNN
 F 1 "74HC32" H 4500 4934 50  0000 C CNN
-F 2 "" H 4500 4700 50  0001 C CNN
+F 2 "Package_SO:SOIC-14_3.9x8.7mm_P1.27mm" H 4500 4700 50  0001 C CNN
 F 3 "http://www.ti.com/lit/gpn/sn74LS32" H 4500 4700 50  0001 C CNN
 	3    4500 4700
@@
 F 0 "U8" H 6800 4025 50  0000 C CNN
 F 1 "74HC86" H 6800 3934 50  0000 C CNN
-F 2 "" H 6800 3700 50  0001 C CNN
+F 2 "Package_SO:SOIC-14_3.9x8.7mm_P1.27mm" H 6800 3700 50  0001 C CNN
 F 3 "http://www.ti.com/lit/gpn/sn74HC86" H 6800 3700 50  0001 C CNN
 	3    6800 3700
@@
 F 0 "U8" H 7750 4225 50  0000 C CNN
 F 1 "74HC86" H 7750 4134 50  0000 C CNN
-F 2 "" H 7750 3900 50  0001 C CNN
+F 2 "Package_SO:SOIC-14_3.9x8.7mm_P1.27mm" H 7750 3900 50  0001 C CNN
 F 3 "http://www.ti.com/lit/gpn/sn74HC86" H 7750 3900 50  0001 C CNN
 	4    7750 3900
@@
 F 0 "U9" H 7750 4775 50  0000 C CNN
 F 1 "74HC08" H 7750 4684 50  0000 C CNN
-F 2 "" H 7750 4450 50  0001 C CNN
+F 2 "Package_SO:SOIC-14_3.9x8.7mm_P1.27mm" H 7750 4450 50  0001 C CNN
 F 3 "http://www.ti.com/lit/gpn/sn74LS08" H 7750 4450 50  0001 C CNN
 	3    7750 4450
@@
 F 0 "U9" H 7750 5375 50  0000 C CNN
 F 1 "74HC08" H 7750 5284 50  0000 C CNN
-F 2 "" H 7750 5050 50  0001 C CNN
+F 2 "Package_SO:SOIC-14_3.9x8.7mm_P1.27mm" H 7750 5050 50  0001 C CNN
 F 3 "http://www.ti.com/lit/gpn/sn74LS08" H 7750 5050 50  0001 C CNN
 	4    7750 5050
@@
 F 0 "U7" H 8500 5075 50  0000 C CNN
 F 1 "74HC32" H 8500 4984 50  0000 C CNN
-F 2 "" H 8500 4750 50  0001 C CNN
+F 2 "Package_SO:SOIC-14_3.9x8.7mm_P1.27mm" H 8500 4750 50  0001 C CNN
 F 3 "http://www.ti.com/lit/gpn/sn74LS32" H 8500 4750 50  0001 C CNN
 	4    8500 4750
@@
 P 1950 1550
 AR Path="/5C594F9A/5C75462B" Ref="#PWR?"  Part="1"
-AR Path="/5C594F14/5C75462B" Ref="#PWR09"  Part="1"
-F 0 "#PWR09" H 1950 1300 50  0001 C CNN
+AR Path="/5C594F14/5C75462B" Ref="#PWR023"  Part="1"
+F 0 "#PWR023" H 1950 1300 50  0001 C CNN
 F 1 "GND" H 1955 1377 50  0000 C CNN
 F 2 "" H 1950 1550 50  0001 C CNN
@@
 P 950 6900
 AR Path="/5C594F9A/5C754641" Ref="C?"  Part="1"
-AR Path="/5C594F14/5C754641" Ref="C5"  Part="1"
-F 0 "C5" H 1065 6946 50  0000 L CNN
+AR Path="/5C594F14/5C754641" Ref="C11"  Part="1"
+F 0 "C11" H 1065 6946 50  0000 L CNN
 F 1 "100n" H 1065 6855 50  0000 L CNN
-F 2 "" H 988 6750 50  0001 C CNN
+F 2 "Capacitor_SMD:C_0805_2012Metric" H 988 6750 50  0001 C CNN
 F 3 "~" H 950 6900 50  0001 C CNN
 	1    950  6900
@@
 P 2150 6900
 AR Path="/5C594F9A/5C754648" Ref="C?"  Part="1"
-AR Path="/5C594F14/5C754648" Ref="C6"  Part="1"
-F 0 "C6" H 2265 6946 50  0000 L CNN
+AR Path="/5C594F14/5C754648" Ref="C12"  Part="1"
+F 0 "C12" H 2265 6946 50  0000 L CNN
 F 1 "100n" H 2265 6855 50  0000 L CNN
-F 2 "" H 2188 6750 50  0001 C CNN
+F 2 "Capacitor_SMD:C_0805_2012Metric" H 2188 6750 50  0001 C CNN
 F 3 "~" H 2150 6900 50  0001 C CNN
 	1    2150 6900
@@
 P 3350 6900
 AR Path="/5C594F9A/5C75464F" Ref="C?"  Part="1"
-AR Path="/5C594F14/5C75464F" Ref="C7"  Part="1"
-F 0 "C7" H 3465 6946 50  0000 L CNN
+AR Path="/5C594F14/5C75464F" Ref="C13"  Part="1"
+F 0 "C13" H 3465 6946 50  0000 L CNN
 F 1 "100n" H 3465 6855 50  0000 L CNN
-F 2 "" H 3388 6750 50  0001 C CNN
+F 2 "Capacitor_SMD:C_0805_2012Metric" H 3388 6750 50  0001 C CNN
 F 3 "~" H 3350 6900 50  0001 C CNN
 	1    3350 6900
@@
 P 4550 6900
 AR Path="/5C594F9A/5C754656" Ref="C?"  Part="1"
-AR Path="/5C594F14/5C754656" Ref="C8"  Part="1"
-F 0 "C8" H 4665 6946 50  0000 L CNN
+AR Path="/5C594F14/5C754656" Ref="C14"  Part="1"
+F 0 "C14" H 4665 6946 50  0000 L CNN
 F 1 "100n" H 4665 6855 50  0000 L CNN
-F 2 "" H 4588 6750 50  0001 C CNN
+F 2 "Capacitor_SMD:C_0805_2012Metric" H 4588 6750 50  0001 C CNN
 F 3 "~" H 4550 6900 50  0001 C CNN
 	1    4550 6900
@@
 P 5750 6900
 AR Path="/5C594F9A/5C75465D" Ref="C?"  Part="1"
-AR Path="/5C594F14/5C75465D" Ref="C9"  Part="1"
-F 0 "C9" H 5865 6946 50  0000 L CNN
+AR Path="/5C594F14/5C75465D" Ref="C15"  Part="1"
+F 0 "C15" H 5865 6946 50  0000 L CNN
 F 1 "100n" H 5865 6855 50  0000 L CNN
-F 2 "" H 5788 6750 50  0001 C CNN
+F 2 "Capacitor_SMD:C_0805_2012Metric" H 5788 6750 50  0001 C CNN
 F 3 "~" H 5750 6900 50  0001 C CNN
 	1    5750 6900
@@
 P 3550 6250
 AR Path="/5C594F9A/5C754664" Ref="#PWR?"  Part="1"
-AR Path="/5C594F14/5C754664" Ref="#PWR010"  Part="1"
-F 0 "#PWR010" H 3550 6100 50  0001 C CNN
+AR Path="/5C594F14/5C754664" Ref="#PWR024"  Part="1"
+F 0 "#PWR024" H 3550 6100 50  0001 C CNN
 F 1 "VCC" H 3567 6423 50  0000 C CNN
 F 2 "" H 3550 6250 50  0001 C CNN
@@
 P 3550 7550
 AR Path="/5C594F9A/5C75466A" Ref="#PWR?"  Part="1"
-AR Path="/5C594F14/5C75466A" Ref="#PWR011"  Part="1"
-F 0 "#PWR011" H 3550 7300 50  0001 C CNN
+AR Path="/5C594F14/5C75466A" Ref="#PWR025"  Part="1"
+F 0 "#PWR025" H 3550 7300 50  0001 C CNN
 F 1 "GND" H 3555 7377 50  0000 C CNN
 F 2 "" H 3550 7550 50  0001 C CNN
