File: core/TD4_core/Multiplexer_4x_4-1.sch (KiCad schematic (older format))
At the start: 4 parts

Commit message: Started refactoring
Connections:
- net In_A_0 renamed A0
- net In_A_1 renamed A1
- net In_A_2 renamed A2
- net In_A_3 renamed A3
- net In_B_0 renamed B0
- net In_B_1 renamed B1
- net In_B_2 renamed B2
- net In_B_3 renamed B3
- net In_IN_0 renamed IN0
- net In_IN_1 renamed IN1
- net In_IN_2 renamed IN2
- net In_IN_3 renamed IN3
- net Out_0: no longer names the net of U?.7 (Za)
- net Out_1: no longer names the net of U?.9 (Zb)
- net Out_2: no longer names the net of U?.7 (Za)
- net Out_3: no longer names the net of U?.9 (Zb)
- net Sel_0 renamed Sel0
- net Sel_1 renamed Sel1
Changed lines of the file:
@@
 EESchema Schematic File Version 4
+LIBS:TD4_core-cache
 EELAYER 26 0
 EELAYER END
@@
 encoding utf-8
 Sheet 5 6
-Title ""
+Title "TD4 core module"
 Date ""
-Rev ""
+Rev "v1.0"
 Comp ""
 Comment1 ""
@@
 	4550 3350 5150 3350
 Text Label 4550 1850 0    50   ~ 0
-In_A_0
+A0
 Text Label 4550 1950 0    50   ~ 0
-In_B_0
+B0
 Text Label 4550 2050 0    50   ~ 0
-In_IN_0
+IN0
+Text Label 4550 3250 0    50   ~ 0
+Sel0
+Text Label 4550 3350 0    50   ~ 0
+Sel1
+Entry Wire Line
+	4450 4800 4550 4900
+Entry Wire Line
+	4450 4900 4550 5000
+Entry Wire Line
+	4450 5000 4550 5100
+Wire Wire Line
+	4550 4900 5150 4900
+Wire Wire Line
+	4550 5000 5150 5000
+Wire Wire Line
+	4550 5100 5150 5100
+Entry Wire Line
+	4450 5500 4550 5600
+Entry Wire Line
+	4450 5600 4550 5700
+Entry Wire Line
+	4450 5700 4550 5800
+Wire Wire Line
+	4550 5600 5150 5600
+Wire Wire Line
+	4550 5700 5150 5700
+Wire Wire Line
+	4550 5800 5150 5800
+Entry Wire Line
+	4450 6200 4550 6300
+Entry Wire Line
+	4450 6300 4550 6400
+Wire Wire Line
+	4550 6300 5150 6300
+Wire Wire Line
+	4550 6400 5150 6400
 Text Label 4550 2550 0    50   ~ 0
-In_A_1
+A1
 Text Label 4550 2650 0    50   ~ 0
-In_B_1
+B1
 Text Label 4550 2750 0    50   ~ 0
-In_IN_1
-Text Label 4550 3250 0    50   ~ 0
-Sel_0
-Text Label 4550 3350 0    50   ~ 0
-Sel_1
-Entry Wire Line
-	4450 4800 4550 4900
-Entry Wire Line
-	4450 4900 4550 5000
-Entry Wire Line
-	4450 5000 4550 5100
-Wire Wire Line
-	4550 4900 5150 4900
-Wire Wire Line
-	4550 5000 5150 5000
-Wire Wire Line
-	4550 5100 5150 5100
-Entry Wire Line
-	4450 5500 4550 5600
-Entry Wire Line
-	4450 5600 4550 5700
-Entry Wire Line
-	4450 5700 4550 5800
-Wire Wire Line
-	4550 5600 5150 5600
-Wire Wire Line
-	4550 5700 5150 5700
-Wire Wire Line
-	4550 5800 5150 5800
-Entry Wire Line
-	4450 6200 4550 6300
-Entry Wire Line
-	4450 6300 4550 6400
-Wire Wire Line
-	4550 6300 5150 6300
-Wire Wire Line
-	4550 6400 5150 6400
+IN1
 Text Label 4550 4900 0    50   ~ 0
-In_A_2
+A2
 Text Label 4550 5000 0    50   ~ 0
-In_B_2
+B2
 Text Label 4550 5100 0    50   ~ 0
-In_IN_2
+IN2
 Text Label 4550 5600 0    50   ~ 0
-In_A_3
+A3
 Text Label 4550 5700 0    50   ~ 0
-In_B_3
+B3
 Text Label 4550 5800 0    50   ~ 0
-In_IN_3
+IN3
 Text Label 4550 6300 0    50   ~ 0
-Sel_0
+Sel0
 Text Label 4550 6400 0    50   ~ 0
-Sel_1
-Wire Bus Line
-	4450 6900 3200 6900
-Entry Wire Line
-	3100 3200 3200 3300
-Entry Wire Line
-	3100 3300 3200 3400
-Entry Wire Line
-	3100 3400 3200 3500
-Entry Wire Line
-	3100 3500 3200 3600
-Entry Wire Line
-	3100 3900 3200 4000
-Entry Wire Line
-	3100 4000 3200 4100
-Entry Wire Line
-	3100 4100 3200 4200
-Entry Wire Line
-	3100 4200 3200 4300
-Entry Wire Line
-	3100 4600 3200 4700
-Entry Wire Line
-	3100 4700 3200 4800
-Entry Wire Line
-	3100 4800 3200 4900
-Entry Wire Line
-	3100 4900 3200 5000
-Entry Wire Line
-	3100 5300 3200 5400
-Entry Wire Line
-	3100 5400 3200 5500
-Wire Wire Line
-	2700 3200 3100 3200
-Wire Wire Line
-	2700 3300 3100 3300
-Wire Wire Line
-	2700 3400 3100 3400
-Wire Wire Line
-	2700 3500 3100 3500
-Text Label 2850 3200 0    50   ~ 0
-In_A_0
-Text Label 2850 3300 0    50   ~ 0
-In_A_1
-Text Label 2850 3400 0    50   ~ 0
-In_A_2
-Text Label 2850 3500 0    50   ~ 0
-In_A_3
-Wire Wire Line
-	2700 3900 3100 3900
-Wire Wire Line
-	2700 4000 3100 4000
-Wire Wire Line
-	2700 4100 3100 4100
-Wire Wire Line
-	2700 4200 3100 4200
-Text Label 2850 3900 0    50   ~ 0
-In_B_0
-Text Label 2850 4000 0    50   ~ 0
-In_B_1
-Text Label 2850 4100 0    50   ~ 0
-In_B_2
-Text Label 2850 4200 0    50   ~ 0
-In_B_3
-Wire Wire Line
-	2700 4600 3100 4600
-Wire Wire Line
-	2700 4700 3100 4700
-Wire Wire Line
-	2700 4800 3100 4800
-Wire Wire Line
-	2700 4900 3100 4900
-Text Label 2850 4600 0    50   ~ 0
-In_IN_0
-Text Label 2850 4700 0    50   ~ 0
-In_IN_1
-Text Label 2850 4800 0    50   ~ 0
-In_IN_2
-Text Label 2850 4900 0    50   ~ 0
-In_IN_3
-Wire Wire Line
-	2700 5300 3100 5300
-Wire Wire Line
-	2700 5400 3100 5400
-Text Label 2850 5300 0    50   ~ 0
-Sel_0
-Text Label 2850 5400 0    50   ~ 0
-Sel_1
-Text HLabel 2700 3200 0    50   Input ~ 0
-In_A_0
-Text HLabel 2700 3300 0    50   Input ~ 0
-In_A_1
-Text HLabel 2700 3400 0    50   Input ~ 0
-In_A_2
-Text HLabel 2700 3500 0    50   Input ~ 0
-In_A_3
-Text HLabel 2700 3900 0    50   Input ~ 0
-In_B_0
-Text HLabel 2700 4000 0    50   Input ~ 0
-In_B_1
-Text HLabel 2700 4100 0    50   Input ~ 0
-In_B_2
-Text HLabel 2700 4200 0    50   Input ~ 0
-In_B_3
-Text HLabel 2700 4600 0    50   Input ~ 0
-In_IN_0
-Text HLabel 2700 4700 0    50   Input ~ 0
-In_IN_1
-Text HLabel 2700 4800 0    50   Input ~ 0
-In_IN_2
-Text HLabel 2700 4900 0    50   Input ~ 0
-In_IN_3
-Text HLabel 2700 5300 0    50   Input ~ 0
-Sel_0
-Text HLabel 2700 5400 0    50   Input ~ 0
-Sel_1
-Wire Wire Line
-	6150 2550 7300 2550
-Wire Wire Line
-	7300 2550 7300 3600
-Wire Wire Line
-	7300 3600 8000 3600
-Wire Wire Line
-	6150 1850 7500 1850
-Wire Wire Line
-	7500 1850 7500 3500
-Wire Wire Line
-	7500 3500 8000 3500
-Wire Wire Line
-	6150 4900 7300 4900
-Wire Wire Line
-	7300 4900 7300 3700
-Wire Wire Line
-	7300 3700 8000 3700
-Wire Wire Line
-	7500 5600 7500 3800
-Wire Wire Line
-	7500 3800 8000 3800
-Wire Wire Line
-	6150 5600 7500 5600
-Wire Bus Line
-	3200 3300 3200 6900
-Wire Bus Line
-	4450 1750 4450 6900
-Text HLabel 8000 3500 2    50   Input ~ 0
-Out_0
-Text HLabel 8000 3600 2    50   Input ~ 0
-Out_1
-Text HLabel 8000 3700 2    50   Input ~ 0
-Out_2
-Text HLabel 8000 3800 2    50   Input ~ 0
-Out_3
+Sel1
 $EndSCHEMATC

Commit message: RAM refactoring goes on
Connections:
- net Q0: now reaches U?.7 (Za)
- net Q1: now reaches U?.9 (Zb)
- net Q2: now reaches U?.7 (Za)
- net Q3: now reaches U?.9 (Zb)
Changed lines of the file:
@@
 	4450 1750 4550 1850
 Entry Wire Line
-	4450 1850 4550 1950
+	4300 1850 4400 1950
 Entry Wire Line
-	4450 1950 4550 2050
+	4150 1950 4250 2050
 Wire Wire Line
 	4550 1850 5150 1850
 Wire Wire Line
-	4550 1950 5150 1950
+	4400 1950 5150 1950
 Wire Wire Line
-	4550 2050 5150 2050
+	4250 2050 5150 2050
 Entry Wire Line
 	4450 2450 4550 2550
 Entry Wire Line
-	4450 2550 4550 2650
+	4300 2550 4400 2650
 Entry Wire Line
-	4450 2650 4550 2750
+	4150 2650 4250 2750
 Wire Wire Line
 	4550 2550 5150 2550
 Wire Wire Line
-	4550 2650 5150 2650
+	4400 2650 5150 2650
 Wire Wire Line
-	4550 2750 5150 2750
+	4250 2750 5150 2750
 Entry Wire Line
-	4450 3150 4550 3250
+	4000 3150 4100 3250
 Entry Wire Line
-	4450 3250 4550 3350
+	4000 3250 4100 3350
 Wire Wire Line
-	4550 3250 5150 3250
+	4100 3250 5150 3250
 Wire Wire Line
-	4550 3350 5150 3350
+	4100 3350 5150 3350
 Text Label 4550 1850 0    50   ~ 0
 A0
@@
 	4450 4800 4550 4900
 Entry Wire Line
-	4450 4900 4550 5000
+	4300 4900 4400 5000
 Entry Wire Line
-	4450 5000 4550 5100
+	4150 5000 4250 5100
 Wire Wire Line
 	4550 4900 5150 4900
 Wire Wire Line
-	4550 5000 5150 5000
+	4400 5000 5150 5000
 Wire Wire Line
-	4550 5100 5150 5100
+	4250 5100 5150 5100
 Entry Wire Line
 	4450 5500 4550 5600
 Entry Wire Line
-	4450 5600 4550 5700
+	4300 5600 4400 5700
 Entry Wire Line
-	4450 5700 4550 5800
+	4150 5700 4250 5800
 Wire Wire Line
 	4550 5600 5150 5600
 Wire Wire Line
-	4550 5700 5150 5700
+	4400 5700 5150 5700
 Wire Wire Line
-	4550 5800 5150 5800
+	4250 5800 5150 5800
 Entry Wire Line
-	4450 6200 4550 6300
+	4000 6200 4100 6300
 Entry Wire Line
-	4450 6300 4550 6400
+	4000 6300 4100 6400
 Wire Wire Line
-	4550 6300 5150 6300
+	4100 6300 5150 6300
 Wire Wire Line
-	4550 6400 5150 6400
+	4100 6400 5150 6400
 Text Label 4550 2550 0    50   ~ 0
 A1
@@
 Text Label 4550 6400 0    50   ~ 0
 Sel1
+Wire Bus Line
+	4450 1300 3400 1300
+Wire Bus Line
+	4300 1500 3400 1500
+Wire Bus Line
+	4150 1700 3400 1700
+Wire Bus Line
+	4000 1900 3400 1900
+Wire Wire Line
+	6150 1850 6400 1850
+Entry Wire Line
+	6400 1850 6500 1950
+Wire Wire Line
+	6150 2550 6400 2550
+Entry Wire Line
+	6400 2550 6500 2650
+Wire Wire Line
+	6150 4900 6400 4900
+Entry Wire Line
+	6400 4900 6500 5000
+Wire Wire Line
+	6150 5600 6400 5600
+Entry Wire Line
+	6400 5600 6500 5700
+Wire Bus Line
+	6500 1300 7300 1300
+Wire Bus Line
+	4000 1900 4000 6300
+Wire Bus Line
+	4150 1700 4150 5700
+Wire Bus Line
+	4300 1500 4300 5600
+Wire Bus Line
+	4450 1300 4450 5500
+Wire Bus Line
+	6500 1300 6500 5700
+Text Label 6350 1850 2    50   ~ 0
+Q0
+Text Label 6350 2550 2    50   ~ 0
+Q1
+Text Label 6350 4900 2    50   ~ 0
+Q2
+Text Label 6350 5600 2    50   ~ 0
+Q3
+Text Label 3500 1300 0    50   ~ 0
+A[0..3]
+Text Label 3500 1500 0    50   ~ 0
+B[0..3]
+Text Label 3500 1700 0    50   ~ 0
+IN[0..3]
+Text Label 3500 1900 0    50   ~ 0
+Sel[0..3]
+Text Label 6950 1300 0    50   ~ 0
+Q[0..3]
+Text HLabel 3400 1300 0    50   Input ~ 0
+A
+Text HLabel 3400 1500 0    50   Input ~ 0
+B
+Text HLabel 3400 1700 0    50   Input ~ 0
+IN
+Text HLabel 3400 1900 0    50   Input ~ 0
+Sel
+Text HLabel 7300 1300 2    50   Output ~ 0
+Q
 $EndSCHEMATC

Commit message: Main core schematic done; only decoder left
Changed lines of the file:
@@
 $Descr A4 11693 8268
 encoding utf-8
-Sheet 5 6
+Sheet 5 9
 Title "TD4 core module"
 Date ""
@@
 Wire Bus Line
 	6500 1300 7300 1300
-Wire Bus Line
-	4000 1900 4000 6300
-Wire Bus Line
-	4150 1700 4150 5700
-Wire Bus Line
-	4300 1500 4300 5600
-Wire Bus Line
-	4450 1300 4450 5500
-Wire Bus Line
-	6500 1300 6500 5700
 Text Label 6350 1850 2    50   ~ 0
 Q0
@@
 IN[0..3]
 Text Label 3500 1900 0    50   ~ 0
-Sel[0..3]
+Sel[0..1]
 Text Label 6950 1300 0    50   ~ 0
 Q[0..3]
 Text HLabel 3400 1300 0    50   Input ~ 0
-A
+A[0..3]
 Text HLabel 3400 1500 0    50   Input ~ 0
-B
+B[0..3]
 Text HLabel 3400 1700 0    50   Input ~ 0
-IN
+IN[0..3]
 Text HLabel 3400 1900 0    50   Input ~ 0
-Sel
+Sel[0..1]
 Text HLabel 7300 1300 2    50   Output ~ 0
-Q
+Q[0..3]
+Wire Bus Line
+	4000 1900 4000 6300
+Wire Bus Line
+	4150 1700 4150 5700
+Wire Bus Line
+	4300 1500 4300 5600
+Wire Bus Line
+	4450 1300 4450 5500
+Wire Bus Line
+	6500 1300 6500 5700
 $EndSCHEMATC

Commit message: Core assembled; decoder left
Parts:
- gave numbers to parts that had none: 4
Changed lines of the file:
@@
 $EndDescr
 $Comp
-L 74xx:74LS153 U?
+L 74xx:74LS153 U10
 U 1 1 5C7644A1
 P 5650 2550
-F 0 "U?" H 5400 3650 50  0000 C CNN
+F 0 "U10" H 5400 3650 50  0000 C CNN
 F 1 "74HC153" H 5350 3550 50  0000 C CNN
 F 2 "" H 5650 2550 50  0001 C CNN
@@
 $EndComp
 $Comp
-L 74xx:74LS153 U?
+L 74xx:74LS153 U11
 U 1 1 5C764537
 P 5650 5600
-F 0 "U?" H 5300 6750 50  0000 C CNN
+F 0 "U11" H 5300 6750 50  0000 C CNN
 F 1 "74HC153" H 5300 6650 50  0000 C CNN
 F 2 "" H 5650 5600 50  0001 C CNN
@@
 $EndComp
 $Comp
-L Device:C C?
+L Device:C C11
 U 1 1 5C764650
 P 5900 4350
-F 0 "C?" H 6015 4396 50  0000 L CNN
+F 0 "C11" H 6015 4396 50  0000 L CNN
 F 1 "100n" H 6015 4305 50  0000 L CNN
 F 2 "" H 5938 4200 50  0001 C CNN
@@
 $EndComp
 $Comp
-L Device:C C?
+L Device:C C10
 U 1 1 5C76468E
 P 5900 1300
-F 0 "C?" H 6015 1346 50  0000 L CNN
+F 0 "C10" H 6015 1346 50  0000 L CNN
 F 1 "100n" H 6015 1255 50  0000 L CNN
 F 2 "" H 5938 1150 50  0001 C CNN
@@
 $EndComp
 $Comp
-L power:GND #PWR?
+L power:GND #PWR0112
 U 1 1 5C7647BF
 P 5900 1450
-F 0 "#PWR?" H 5900 1200 50  0001 C CNN
+F 0 "#PWR0112" H 5900 1200 50  0001 C CNN
 F 1 "GND" H 5905 1277 50  0000 C CNN
 F 2 "" H 5900 1450 50  0001 C CNN
@@
 $EndComp
 $Comp
-L power:GND #PWR?
+L power:GND #PWR0113
 U 1 1 5C7647DD
 P 5900 4500
-F 0 "#PWR?" H 5900 4250 50  0001 C CNN
+F 0 "#PWR0113" H 5900 4250 50  0001 C CNN
 F 1 "GND" H 5905 4327 50  0000 C CNN
 F 2 "" H 5900 4500 50  0001 C CNN
@@
 $EndComp
 $Comp
-L power:GND #PWR?
+L power:GND #PWR0114
 U 1 1 5C764814
 P 5650 3650
-F 0 "#PWR?" H 5650 3400 50  0001 C CNN
+F 0 "#PWR0114" H 5650 3400 50  0001 C CNN
 F 1 "GND" H 5655 3477 50  0000 C CNN
 F 2 "" H 5650 3650 50  0001 C CNN
@@
 $EndComp
 $Comp
-L power:GND #PWR?
+L power:GND #PWR0115
 U 1 1 5C764827
 P 5650 6700
-F 0 "#PWR?" H 5650 6450 50  0001 C CNN
+F 0 "#PWR0115" H 5650 6450 50  0001 C CNN
 F 1 "GND" H 5655 6527 50  0000 C CNN
 F 2 "" H 5650 6700 50  0001 C CNN
@@
 $EndComp
 $Comp
-L power:VCC #PWR?
+L power:VCC #PWR0116
 U 1 1 5C764910
 P 5650 4100
-F 0 "#PWR?" H 5650 3950 50  0001 C CNN
+F 0 "#PWR0116" H 5650 3950 50  0001 C CNN
 F 1 "VCC" H 5667 4273 50  0000 C CNN
 F 2 "" H 5650 4100 50  0001 C CNN
@@
 	5650 4150 5650 4600
 $Comp
-L power:VCC #PWR?
+L power:VCC #PWR0117
 U 1 1 5C764973
 P 5650 1050
-F 0 "#PWR?" H 5650 900 50  0001 C CNN
+F 0 "#PWR0117" H 5650 900 50  0001 C CNN
 F 1 "VCC" H 5667 1223 50  0000 C CNN
 F 2 "" H 5650 1050 50  0001 C CNN
@@
 	5050 2350 5150 2350
 $Comp
-L power:GND #PWR?
+L power:GND #PWR0118
 U 1 1 5C7653EA
 P 4950 2300
-F 0 "#PWR?" H 4950 2050 50  0001 C CNN
+F 0 "#PWR0118" H 4950 2050 50  0001 C CNN
 F 1 "GND" H 4955 2127 50  0000 C CNN
 F 2 "" H 4950 2300 50  0001 C CNN
@@
 	5050 2250 5050 2350
 $Comp
-L power:GND #PWR?
+L power:GND #PWR0119
 U 1 1 5C76556D
 P 4950 3000
-F 0 "#PWR?" H 4950 2750 50  0001 C CNN
+F 0 "#PWR0119" H 4950 2750 50  0001 C CNN
 F 1 "GND" H 4955 2827 50  0000 C CNN
 F 2 "" H 4950 3000 50  0001 C CNN
@@
 	5050 5400 5150 5400
 $Comp
-L power:GND #PWR?
+L power:GND #PWR0120
 U 1 1 5C765F00
 P 4950 5350
-F 0 "#PWR?" H 4950 5100 50  0001 C CNN
+F 0 "#PWR0120" H 4950 5100 50  0001 C CNN
 F 1 "GND" H 4955 5177 50  0000 C CNN
 F 2 "" H 4950 5350 50  0001 C CNN
@@
 	5050 5300 5050 5400
 $Comp
-L power:GND #PWR?
+L power:GND #PWR0121
 U 1 1 5C765F0A
 P 4950 6050
-F 0 "#PWR?" H 4950 5800 50  0001 C CNN
+F 0 "#PWR0121" H 4950 5800 50  0001 C CNN
 F 1 "GND" H 4955 5877 50  0000 C CNN
 F 2 "" H 4950 6050 50  0001 C CNN

Commit message: Decoder done (finally!)
Parts:
- renumbered C10 to C29, C11 to C30, U10 to U29, U11 to U30
Changed lines of the file:
@@
 $Descr A4 11693 8268
 encoding utf-8
-Sheet 5 9
+Sheet 5 23
 Title "TD4 core module"
 Date ""
@@
 $EndDescr
 $Comp
-L 74xx:74LS153 U10
+L 74xx:74LS153 U29
 U 1 1 5C7644A1
 P 5650 2550
-F 0 "U10" H 5400 3650 50  0000 C CNN
+F 0 "U29" H 5400 3650 50  0000 C CNN
 F 1 "74HC153" H 5350 3550 50  0000 C CNN
 F 2 "" H 5650 2550 50  0001 C CNN
@@
 $EndComp
 $Comp
-L 74xx:74LS153 U11
+L 74xx:74LS153 U30
 U 1 1 5C764537
 P 5650 5600
-F 0 "U11" H 5300 6750 50  0000 C CNN
+F 0 "U30" H 5300 6750 50  0000 C CNN
 F 1 "74HC153" H 5300 6650 50  0000 C CNN
 F 2 "" H 5650 5600 50  0001 C CNN
@@
 $EndComp
 $Comp
-L Device:C C11
+L Device:C C30
 U 1 1 5C764650
 P 5900 4350
-F 0 "C11" H 6015 4396 50  0000 L CNN
+F 0 "C30" H 6015 4396 50  0000 L CNN
 F 1 "100n" H 6015 4305 50  0000 L CNN
 F 2 "" H 5938 4200 50  0001 C CNN
@@
 $EndComp
 $Comp
-L Device:C C10
+L Device:C C29
 U 1 1 5C76468E
 P 5900 1300
-F 0 "C10" H 6015 1346 50  0000 L CNN
+F 0 "C29" H 6015 1346 50  0000 L CNN
 F 1 "100n" H 6015 1255 50  0000 L CNN
 F 2 "" H 5938 1150 50  0001 C CNN
@@
 $EndComp
 $Comp
-L power:GND #PWR0112
+L power:GND #PWR092
 U 1 1 5C7647BF
 P 5900 1450
-F 0 "#PWR0112" H 5900 1200 50  0001 C CNN
+F 0 "#PWR092" H 5900 1200 50  0001 C CNN
 F 1 "GND" H 5905 1277 50  0000 C CNN
 F 2 "" H 5900 1450 50  0001 C CNN
@@
 $EndComp
 $Comp
-L power:GND #PWR0113
+L power:GND #PWR097
 U 1 1 5C7647DD
 P 5900 4500
-F 0 "#PWR0113" H 5900 4250 50  0001 C CNN
+F 0 "#PWR097" H 5900 4250 50  0001 C CNN
 F 1 "GND" H 5905 4327 50  0000 C CNN
 F 2 "" H 5900 4500 50  0001 C CNN
@@
 $EndComp
 $Comp
-L power:GND #PWR0114
+L power:GND #PWR095
 U 1 1 5C764814
 P 5650 3650
-F 0 "#PWR0114" H 5650 3400 50  0001 C CNN
+F 0 "#PWR095" H 5650 3400 50  0001 C CNN
 F 1 "GND" H 5655 3477 50  0000 C CNN
 F 2 "" H 5650 3650 50  0001 C CNN
@@
 $EndComp
 $Comp
-L power:GND #PWR0115
+L power:GND #PWR0100
 U 1 1 5C764827
 P 5650 6700
-F 0 "#PWR0115" H 5650 6450 50  0001 C CNN
+F 0 "#PWR0100" H 5650 6450 50  0001 C CNN
 F 1 "GND" H 5655 6527 50  0000 C CNN
 F 2 "" H 5650 6700 50  0001 C CNN
@@
 $EndComp
 $Comp
-L power:VCC #PWR0116
+L power:VCC #PWR096
 U 1 1 5C764910
 P 5650 4100
-F 0 "#PWR0116" H 5650 3950 50  0001 C CNN
+F 0 "#PWR096" H 5650 3950 50  0001 C CNN
 F 1 "VCC" H 5667 4273 50  0000 C CNN
 F 2 "" H 5650 4100 50  0001 C CNN
@@
 	5650 4150 5650 4600
 $Comp
-L power:VCC #PWR0117
+L power:VCC #PWR091
 U 1 1 5C764973
 P 5650 1050
-F 0 "#PWR0117" H 5650 900 50  0001 C CNN
+F 0 "#PWR091" H 5650 900 50  0001 C CNN
 F 1 "VCC" H 5667 1223 50  0000 C CNN
 F 2 "" H 5650 1050 50  0001 C CNN
@@
 	5050 2350 5150 2350
 $Comp
-L power:GND #PWR0118
+L power:GND #PWR093
 U 1 1 5C7653EA
 P 4950 2300
-F 0 "#PWR0118" H 4950 2050 50  0001 C CNN
+F 0 "#PWR093" H 4950 2050 50  0001 C CNN
 F 1 "GND" H 4955 2127 50  0000 C CNN
 F 2 "" H 4950 2300 50  0001 C CNN
@@
 	5050 2250 5050 2350
 $Comp
-L power:GND #PWR0119
+L power:GND #PWR094
 U 1 1 5C76556D
 P 4950 3000
-F 0 "#PWR0119" H 4950 2750 50  0001 C CNN
+F 0 "#PWR094" H 4950 2750 50  0001 C CNN
 F 1 "GND" H 4955 2827 50  0000 C CNN
 F 2 "" H 4950 3000 50  0001 C CNN
@@
 	5050 5400 5150 5400
 $Comp
-L power:GND #PWR0120
+L power:GND #PWR098
 U 1 1 5C765F00
 P 4950 5350
-F 0 "#PWR0120" H 4950 5100 50  0001 C CNN
+F 0 "#PWR098" H 4950 5100 50  0001 C CNN
 F 1 "GND" H 4955 5177 50  0000 C CNN
 F 2 "" H 4950 5350 50  0001 C CNN
@@
 	5050 5300 5050 5400
 $Comp
-L power:GND #PWR0121
+L power:GND #PWR099
 U 1 1 5C765F0A
 P 4950 6050
-F 0 "#PWR0121" H 4950 5800 50  0001 C CNN
+F 0 "#PWR099" H 4950 5800 50  0001 C CNN
 F 1 "GND" H 4955 5877 50  0000 C CNN
 F 2 "" H 4950 6050 50  0001 C CNN

Commit message: Core schematic done. Backplane connector added, including separate .sch file to append.
Parts:
- C35: renamed from C29; footprint (none) -> Capacitor_SMD:C_0805_2012Metric
- C36: renamed from C30; footprint (none) -> Capacitor_SMD:C_0805_2012Metric
- U29, U30: footprint (none) -> Package_SO:SOIC-16_3.9x9.9mm_P1.27mm
Changed lines of the file:
@@
 F 0 "U29" H 5400 3650 50  0000 C CNN
 F 1 "74HC153" H 5350 3550 50  0000 C CNN
-F 2 "" H 5650 2550 50  0001 C CNN
+F 2 "Package_SO:SOIC-16_3.9x9.9mm_P1.27mm" H 5650 2550 50  0001 C CNN
 F 3 "http://www.ti.com/lit/gpn/sn74LS153" H 5650 2550 50  0001 C CNN
 	1    5650 2550
@@
 F 0 "U30" H 5300 6750 50  0000 C CNN
 F 1 "74HC153" H 5300 6650 50  0000 C CNN
-F 2 "" H 5650 5600 50  0001 C CNN
+F 2 "Package_SO:SOIC-16_3.9x9.9mm_P1.27mm" H 5650 5600 50  0001 C CNN
 F 3 "http://www.ti.com/lit/gpn/sn74LS153" H 5650 5600 50  0001 C CNN
 	1    5650 5600
@@
 $EndComp
 $Comp
-L Device:C C30
+L Device:C C36
 U 1 1 5C764650
 P 5900 4350
-F 0 "C30" H 6015 4396 50  0000 L CNN
+F 0 "C36" H 6015 4396 50  0000 L CNN
 F 1 "100n" H 6015 4305 50  0000 L CNN
-F 2 "" H 5938 4200 50  0001 C CNN
+F 2 "Capacitor_SMD:C_0805_2012Metric" H 5938 4200 50  0001 C CNN
 F 3 "~" H 5900 4350 50  0001 C CNN
 	1    5900 4350
@@
 $EndComp
 $Comp
-L Device:C C29
+L Device:C C35
 U 1 1 5C76468E
 P 5900 1300
-F 0 "C29" H 6015 1346 50  0000 L CNN
+F 0 "C35" H 6015 1346 50  0000 L CNN
 F 1 "100n" H 6015 1255 50  0000 L CNN
-F 2 "" H 5938 1150 50  0001 C CNN
+F 2 "Capacitor_SMD:C_0805_2012Metric" H 5938 1150 50  0001 C CNN
 F 3 "~" H 5900 1300 50  0001 C CNN
 	1    5900 1300
@@
 $EndComp
 $Comp
-L power:GND #PWR092
+L power:GND #PWR0106
 U 1 1 5C7647BF
 P 5900 1450
-F 0 "#PWR092" H 5900 1200 50  0001 C CNN
+F 0 "#PWR0106" H 5900 1200 50  0001 C CNN
 F 1 "GND" H 5905 1277 50  0000 C CNN
 F 2 "" H 5900 1450 50  0001 C CNN
@@
 $EndComp
 $Comp
-L power:GND #PWR097
+L power:GND #PWR0111
 U 1 1 5C7647DD
 P 5900 4500
-F 0 "#PWR097" H 5900 4250 50  0001 C CNN
+F 0 "#PWR0111" H 5900 4250 50  0001 C CNN
 F 1 "GND" H 5905 4327 50  0000 C CNN
 F 2 "" H 5900 4500 50  0001 C CNN
@@
 $EndComp
 $Comp
-L power:GND #PWR095
+L power:GND #PWR0109
 U 1 1 5C764814
 P 5650 3650
-F 0 "#PWR095" H 5650 3400 50  0001 C CNN
+F 0 "#PWR0109" H 5650 3400 50  0001 C CNN
 F 1 "GND" H 5655 3477 50  0000 C CNN
 F 2 "" H 5650 3650 50  0001 C CNN
@@
 $EndComp
 $Comp
-L power:GND #PWR0100
+L power:GND #PWR0114
 U 1 1 5C764827
 P 5650 6700
-F 0 "#PWR0100" H 5650 6450 50  0001 C CNN
+F 0 "#PWR0114" H 5650 6450 50  0001 C CNN
 F 1 "GND" H 5655 6527 50  0000 C CNN
 F 2 "" H 5650 6700 50  0001 C CNN
@@
 $EndComp
 $Comp
-L power:VCC #PWR096
+L power:VCC #PWR0110
 U 1 1 5C764910
 P 5650 4100
-F 0 "#PWR096" H 5650 3950 50  0001 C CNN
+F 0 "#PWR0110" H 5650 3950 50  0001 C CNN
 F 1 "VCC" H 5667 4273 50  0000 C CNN
 F 2 "" H 5650 4100 50  0001 C CNN
@@
 	5650 4150 5650 4600
 $Comp
-L power:VCC #PWR091
+L power:VCC #PWR0105
 U 1 1 5C764973
 P 5650 1050
-F 0 "#PWR091" H 5650 900 50  0001 C CNN
+F 0 "#PWR0105" H 5650 900 50  0001 C CNN
 F 1 "VCC" H 5667 1223 50  0000 C CNN
 F 2 "" H 5650 1050 50  0001 C CNN
@@
 	5050 2350 5150 2350
 $Comp
-L power:GND #PWR093
+L power:GND #PWR0107
 U 1 1 5C7653EA
 P 4950 2300
-F 0 "#PWR093" H 4950 2050 50  0001 C CNN
+F 0 "#PWR0107" H 4950 2050 50  0001 C CNN
 F 1 "GND" H 4955 2127 50  0000 C CNN
 F 2 "" H 4950 2300 50  0001 C CNN
@@
 	5050 2250 5050 2350
 $Comp
-L power:GND #PWR094
+L power:GND #PWR0108
 U 1 1 5C76556D
 P 4950 3000
-F 0 "#PWR094" H 4950 2750 50  0001 C CNN
+F 0 "#PWR0108" H 4950 2750 50  0001 C CNN
 F 1 "GND" H 4955 2827 50  0000 C CNN
 F 2 "" H 4950 3000 50  0001 C CNN
@@
 	5050 5400 5150 5400
 $Comp
-L power:GND #PWR098
+L power:GND #PWR0112
 U 1 1 5C765F00
 P 4950 5350
-F 0 "#PWR098" H 4950 5100 50  0001 C CNN
+F 0 "#PWR0112" H 4950 5100 50  0001 C CNN
 F 1 "GND" H 4955 5177 50  0000 C CNN
 F 2 "" H 4950 5350 50  0001 C CNN
@@
 	5050 5300 5050 5400
 $Comp
-L power:GND #PWR099
+L power:GND #PWR0113
 U 1 1 5C765F0A
 P 4950 6050
-F 0 "#PWR099" H 4950 5800 50  0001 C CNN
+F 0 "#PWR0113" H 4950 5800 50  0001 C CNN
 F 1 "GND" H 4955 5877 50  0000 C CNN
 F 2 "" H 4950 6050 50  0001 C CNN
