File: core/TD4_core/Decoder.sch (KiCad schematic (older format))
At the start: 0 parts

Commit message: Decoder done (finally!)
Parts:
- added C10, C11, C12, C13, C14, C15: 100n, symbol Device:C
- added U10: 74LS151, symbol 74xx:74LS151
- added U11, U12, U14: 74AHC1G04, symbol 74xGxx:74AHC1G04
- added U13, U15: 74AHC1G86, symbol 74xGxx:74AHC1G86
Connections:
- new net: U10.7 (~E), U11.4
- new net 3state_e: U12.2, U13.2
- new net C: U10.13 (I6)
- new net GND: C10.1, C11.2, C12.2, C13.2, C14.2, C15.2, U10.1 (I3), U10.12 (I7), U10.15 (I4), U10.3 (I1), U10.8 (GND), U11.3 (GND), U12.3 (GND), U13.3 (GND), U14.3 (GND), U15.3 (GND)
- new net Instr0: U10.11 (S0), U15.1
- new net Instr1: U10.10 (S1)
- new net Instr2: U10.9 (S2), U13.1
- new net Instr3: U11.2
- new net RAM_RW: U12.4
- new net RAM_WE: U14.4
- new net VCC: C10.2, C11.1, C12.1, C13.1, C14.1, C15.1, U10.14 (I5), U10.16 (VCC), U10.2 (I2), U10.4 (I0), U11.5 (VCC), U12.5 (VCC), U13.5 (VCC), U14.5 (VCC), U15.5 (VCC)
- new net dst_sel0: U13.4
- new net r_sel_e: U10.5 (Z)
- new net sheet5C66DD7A/Q1: U14.2
- new net sheet5C67666E/Q0: U15.2
- new net src_sel0: U15.4
- no-connect marks 0 -> 2
Other:
- note added: "Comparators"

Commit message: Core schematic done. Backplane connector added, including separate .sch file to append.
Parts:
- C16: renamed from C10; footprint (none) -> Capacitor_SMD:C_0805_2012Metric
- C17: renamed from C11; footprint (none) -> Capacitor_SMD:C_0805_2012Metric
- C18: renamed from C12; footprint (none) -> Capacitor_SMD:C_0805_2012Metric
- C19: renamed from C13; footprint (none) -> Capacitor_SMD:C_0805_2012Metric
- C20: renamed from C14; footprint (none) -> Capacitor_SMD:C_0805_2012Metric
- C21: renamed from C15; footprint (none) -> Capacitor_SMD:C_0805_2012Metric
- U10: footprint (none) -> Package_SO:SOIC-16_3.9x9.9mm_P1.27mm
- U11, U12, U13, U14, U15: footprint (none) -> Package_TO_SOT_SMD:SOT-23-5

Commit message: ROM routing done
Parts:
- U10: value 74LS151 -> 74HC151
Changed lines of the file:
@@
 P 10000 2400
 F 0 "U10" H 9700 3500 50  0000 C CNN
-F 1 "74LS151" H 9700 3400 50  0000 C CNN
+F 1 "74HC151" H 9700 3400 50  0000 C CNN
 F 2 "Package_SO:SOIC-16_3.9x9.9mm_P1.27mm" H 10000 2400 50  0001 C CNN
 F 3 "http://www.ti.com/lit/gpn/sn74LS151" H 10000 2400 50  0001 C CNN
